File: m3psu/pcb/file56E22DB2.sch (KiCad schematic (older format))
At the start: 6 parts

Commit message: Changes to Li-ion charger, north local interconnect.
Changed lines of the file:
@@
 	5100 3300 5100 3450
 Wire Wire Line
-	5100 3550 5100 3700
-Wire Wire Line
-	5100 3700 5100 3750
+	5100 3550 5100 3750
 Wire Wire Line
 	5100 3700 5300 3700
@@
 	5500 4050 5500 4150
 Wire Wire Line
-	5100 3300 5500 3300
-Wire Wire Line
-	5500 3300 5700 3300
+	5100 3300 5700 3300
 Wire Wire Line
 	5500 4450 5500 4500

Commit message: Grouped components, sorted internal interconnects. Sheets size now roughly proportional to number of components inside.
Parts:
- Q? (x2): Farnell 2364070 -> 2490619
Changed lines of the file:
@@
 $Descr A4 11693 8268
 encoding utf-8
-Sheet 13 13
+Sheet 13 14
 Title ""
 Date ""
@@
 F 2 "" H 5500 4250 50  0001 C CNN
 F 3 "" H 5500 4250 50  0001 C CNN
-F 4 "2364070" H 5500 4250 60  0001 C CNN "Farnell"
+F 4 "2490619" H 5500 4250 60  0001 C CNN "Farnell"
 	1    5500 4250
 	1    0    0    -1
@@
 F 2 "" H 5100 3850 50  0001 C CNN
 F 3 "" H 5100 3850 50  0001 C CNN
-F 4 "2364070" H 5100 3850 60  0001 C CNN "Farnell"
+F 4 "2490619" H 5100 3850 60  0001 C CNN "Farnell"
 	1    5100 3850
 	1    0    0    -1
