File: m3dl/strain_1-3/strain_1-3.sch (KiCad schematic (older format))
At the start: 66 parts, among them IC1 AD8226, IC2 AD8541, IC3 AD8226, IC4 AD8541, IC5 AD8656, IC6 AD8226, IC7 AD8541, IC8 AD8656, IC9 AD8656, J1 WEST TOP, J2 EAST TOP, J3 WEST BOT, J4 EAST BOT, J5 SOUTH TOP, J6 SOUTH BOT, J7 S1, J8 S3, J9 S2

Commit message: Modifications as per review document
Parts:
- added C22, C23, C24, C25, C26, C27, C28, C29, C30, C31, C32, C33: 100n, agg:0603-L, symbol C_Small
- added C34: 10u, agg:0603-L, symbol C_Small
- added D1, D2, D3, D4, D5, D6, D7, D8, D9: ESD_DIODE, agg:0402, symbol ESD_DIODE
- added R28, R29, R30: 0R, agg:0603, symbol R
Connections:
- net 3v3: now also C23.1, C24.1, C25.1, C27.1, C28.1, C29.1, C31.1, C32.1, C33.1, C34.1, D3.2, D6.2, D9.2
- net GND: now also C22.2, C23.2, C24.2, C25.2, C26.2, C27.2, C28.2, C29.2, C30.2, C31.2, C32.2, C33.2, C34.2, D1.1, D2.1, D3.1, D4.1, D5.1, D6.1, D7.1, D8.1, D9.1
- net STRAIN1+: now also D2.2
- net STRAIN1-: now also D1.2
- net STRAIN2+: now also D5.2
- net STRAIN2-: now also D4.2
- net STRAIN3+: now also D8.2
- net STRAIN3-: now also D7.2
- net at C4.2, C5.1, IC3.1 (-IN)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: now also R28.1
- net at IC4.3 (+), R7.1, R8.2: now also C22.1, R28.2
- net at C15.2, C16.1, IC6.1 (-IN)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: now also R30.1
- net at IC7.3 (+), R21.1, R22.2: now also C30.1, R30.2
- net at C1.2, C2.1, IC1.1 (-IN)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: now also R29.1
- net at IC2.3 (+), R5.1, R6.2: now also C26.1, R29.2
Other:
- note removed: "N.B. We require 2x copies of this board, one as shown and one \nwhere Strain 1 - 3 are connected to Strain 4 - 6 respectivly. \nWe will generate the gerbers for the first and then make a slight \nmodification to the netlist in order to generate the second."
- moved on the sheet: J7, J9

Commit message: Added current limiting functionality
Parts:
- added C35, C37: 1u, agg:0402-L, symbol C_Small
- added C36: 100n, agg:0402-L, symbol C_Small
- added IC10: NCP380, agg:DFN-6-EP-ONSEMI, symbol NCP380
- added R31: 10k, agg:0402-L, symbol R
- added R32: 110k, agg:0402-L, symbol R
Connections:
- net 3v3: now also C37.1, IC10.1 (OUT); no longer J1.11, J3.11
- net GND: now also C35.2, C36.2, C37.2, IC10.5 (GND), IC10.EP (GND), R32.2
- new net: IC10.2 (ILIM), R32.1
- new net: C36.1, IC10.4 (~EN), R31.2
- new net 3v3_DL: C35.1, IC10.6 (IN), J1.11, J3.11, R31.1
- no-connect marks 0 -> 1
Other:
- note added: "CURRENT LIMITING:"
- note removed: "Working Voltage"
Changed lines of the file:
@@
 L 3v3 #PWR023
 U 1 1 56CAA54D
-P 15400 10200
-F 0 "#PWR023" H 15400 10310 50  0001 L CNN
-F 1 "3v3" H 15400 10290 50  0000 C CNN
-F 2 "" H 15400 10200 60  0000 C CNN
-F 3 "" H 15400 10200 60  0000 C CNN
-	1    15400 10200
-	1    0    0    -1
-$EndComp
-Text Label 15550 10300 0    60   ~ 0
+P 11050 4400
+F 0 "#PWR023" H 11050 4510 50  0001 L CNN
+F 1 "3v3" H 11050 4490 50  0000 C CNN
+F 2 "" H 11050 4400 60  0000 C CNN
+F 3 "" H 11050 4400 60  0000 C CNN
+	1    11050 4400
+	1    0    0    -1
+$EndComp
+Text Label 9150 4450 2    60   ~ 0
 3v3_DL
-Text Notes 15250 10500 0    60   ~ 0
-Working Voltage
 $Comp
 L AD8226 IC3
@@
 	1700 1550 1550 1550
 Wire Wire Line
-	15400 10200 15400 10300
-Wire Wire Line
-	15400 10300 15550 10300
-Wire Notes Line
-	15900 10050 15900 10350
-Wire Notes Line
-	15900 10350 15300 10350
-Wire Notes Line
-	15300 10350 15300 10050
-Wire Notes Line
-	15300 10050 15900 10050
-Wire Wire Line
 	2100 1350 2550 1350
 Wire Wire Line
@@
 	8250 500  8250 6300
 Wire Notes Line
-	500  6300 10200 6300
+	500  6300 12500 6300
 Wire Notes Line
 	10200 6300 10200 8500
@@
 	14550 2750 14550 2500
 Connection ~ 14550 2500
+$Comp
+L C_Small C35
+U 1 1 5761B451
+P 9250 4800
+F 0 "C35" H 9260 4870 50  0000 L CNN
+F 1 "1u" H 9260 4720 50  0000 L CNN
+F 2 "agg:0402-L" H 9250 4800 50  0001 C CNN
+F 3 "" H 9250 4800 50  0000 C CNN
+	1    9250 4800
+	-1   0    0    -1
+$EndComp
+$Comp
+L C_Small C37
+U 1 1 5761CF5B
+P 11350 4800
+F 0 "C37" H 11360 4870 50  0000 L CNN
+F 1 "1u" H 11360 4720 50  0000 L CNN
+F 2 "agg:0402-L" H 11350 4800 50  0001 C CNN
+F 3 "" H 11350 4800 50  0000 C CNN
+	1    11350 4800
+	1    0    0    -1
+$EndComp
+$Comp
+L C_Small C36
+U 1 1 5761D0AF
+P 9850 4800
+F 0 "C36" H 9860 4870 50  0000 L CNN
+F 1 "100n" H 9860 4720 50  0000 L CNN
+F 2 "agg:0402-L" H 9850 4800 50  0001 C CNN
+F 3 "" H 9850 4800 50  0000 C CNN
+	1    9850 4800
+	1    0    0    -1
+$EndComp
+$Comp
+L R R32
+U 1 1 5761F126
+P 11050 4900
+F 0 "R32" V 10950 4900 50  0000 C CNN
+F 1 "110k" V 11050 4900 39  0000 C CNN
+F 2 "agg:0402-L" V 10980 4900 50  0001 C CNN
+F 3 "" H 11050 4900 50  0000 C CNN
+	1    11050 4900
+	-1   0    0    -1
+$EndComp
+$Comp
+L R R31
+U 1 1 57620D71
+P 9650 4650
+F 0 "R31" V 9550 4650 50  0000 C CNN
+F 1 "10k" V 9650 4650 39  0000 C CNN
+F 2 "agg:0402-L" V 9580 4650 50  0001 C CNN
+F 3 "" H 9650 4650 50  0000 C CNN
+	1    9650 4650
+	0    -1   1    0
+$EndComp
+Wire Wire Line
+	9800 4650 10150 4650
+Wire Wire Line
+	9850 4650 9850 4700
+$Comp
+L GND #PWR0102
+U 1 1 57624A54
+P 10100 5150
+F 0 "#PWR0102" H 10100 4900 50  0001 C CNN
+F 1 "GND" H 10100 5000 50  0000 C CNN
+F 2 "" H 10100 5150 50  0000 C CNN
+F 3 "" H 10100 5150 50  0000 C CNN
+	1    10100 5150
+	1    0    0    -1
+$EndComp
+$Comp
+L NCP380 IC10
+U 1 1 57604F3C
+P 10550 4750
+F 0 "IC10" H 10250 5150 50  0000 L CNN
+F 1 "NCP380" H 10250 4350 50  0000 L CNN
+F 2 "agg:DFN-6-EP-ONSEMI" H 10250 4250 50  0001 L CNN
+F 3 "http://www.onsemi.com/pub_link/Collateral/NCP380-D.PDF" H 10250 4150 50  0001 L CNN
+F 4 "2464412" H 10250 4050 50  0001 L CNN "Farnell"
+	1    10550 4750
+	1    0    0    -1
+$EndComp
+Wire Wire Line
+	10150 5050 10100 5050
+Wire Wire Line
+	10100 4950 10100 5150
+Wire Wire Line
+	10150 4950 10100 4950
+Connection ~ 10100 5050
+$Comp
+L GND #PWR0103
+U 1 1 5760F261
+P 11050 5150
+F 0 "#PWR0103" H 11050 4900 50  0001 C CNN
+F 1 "GND" H 11050 5000 50  0000 C CNN
+F 2 "" H 11050 5150 50  0000 C CNN
+F 3 "" H 11050 5150 50  0000 C CNN
+	1    11050 5150
+	1    0    0    -1
+$EndComp
+$Comp
+L 3v3 #PWR0104
+U 1 1 5760F398
+P 11350 4400
+F 0 "#PWR0104" H 11350 4510 50  0001 L CNN
+F 1 "3v3" H 11350 4490 50  0000 C CNN
+F 2 "" H 11350 4400 60  0000 C CNN
+F 3 "" H 11350 4400 60  0000 C CNN
+	1    11350 4400
+	1    0    0    -1
+$EndComp
+$Comp
+L GND #PWR0105
+U 1 1 5760F4CF
+P 11350 5150
+F 0 "#PWR0105" H 11350 4900 50  0001 C CNN
+F 1 "GND" H 11350 5000 50  0000 C CNN
+F 2 "" H 11350 5150 50  0000 C CNN
+F 3 "" H 11350 5150 50  0000 C CNN
+	1    11350 5150
+	1    0    0    -1
+$EndComp
+Wire Wire Line
+	11350 4700 11350 4400
+Wire Wire Line
+	11350 4900 11350 5150
+Wire Wire Line
+	10950 4650 11050 4650
+Wire Wire Line
+	11050 4650 11050 4750
+Wire Wire Line
+	11050 5050 11050 5150
+NoConn ~ 10150 4750
+Wire Wire Line
+	10950 4450 11050 4450
+Wire Wire Line
+	11050 4450 11050 4400
+Wire Wire Line
+	9150 4450 10150 4450
+Connection ~ 9850 4650
+Wire Wire Line
+	9450 4650 9500 4650
+Wire Wire Line
+	9450 4400 9450 4650
+Connection ~ 9450 4450
+Wire Wire Line
+	9850 4900 9850 5150
+$Comp
+L GND #PWR0106
+U 1 1 5761682A
+P 9850 5150
+F 0 "#PWR0106" H 9850 4900 50  0001 C CNN
+F 1 "GND" H 9850 5000 50  0000 C CNN
+F 2 "" H 9850 5150 50  0000 C CNN
+F 3 "" H 9850 5150 50  0000 C CNN
+	1    9850 5150
+	1    0    0    -1
+$EndComp
+Wire Wire Line
+	9250 4700 9250 4450
+Connection ~ 9250 4450
+Wire Wire Line
+	9250 4900 9250 5150
+$Comp
+L GND #PWR0107
+U 1 1 57616F25
+P 9250 5150
+F 0 "#PWR0107" H 9250 4900 50  0001 C CNN
+F 1 "GND" H 9250 5000 50  0000 C CNN
+F 2 "" H 9250 5150 50  0000 C CNN
+F 3 "" H 9250 5150 50  0000 C CNN
+	1    9250 5150
+	1    0    0    -1
+$EndComp
+Wire Notes Line
+	12500 6300 12500 3400
+Text Notes 10150 3800 2    118  ~ 24
+CURRENT LIMITING:
+$Comp
+L PWR #FLG0108
+U 1 1 57621F44
+P 9450 4400
+F 0 "#FLG0108" H 9450 4560 50  0001 C CNN
+F 1 "PWR" H 9450 4490 50  0000 C CNN
+F 2 "" H 9450 4400 50  0001 C CNN
+F 3 "" H 9450 4400 50  0001 C CNN
+	1    9450 4400
+	1    0    0    -1
+$EndComp
 $EndSCHEMATC

Commit message: Finalised BOM
Parts:
- C1, C15, C17, C3, C4, C6: Farnell (none) -> 1813443
- C10, C13, C14, C19, C21, C9: Farnell (none) -> 1865539
- C11, C12, C18, C20, C7, C8: Farnell (none) -> 1865464
- C16, C2, C5: Farnell (none) -> 1457729
- C22, C23, C24, C25, C26, C27, C28, C29, C30, C31, C32, C33: Farnell (none) -> 2496834
- C34: Farnell (none) -> 2211164
- C35, C37: Farnell (none) -> 2346884
- C36: Farnell (none) -> 2496771
- J7, J8, J9: RS (none) -> 279-9285
- R1, R19, R2, R20, R3, R4: Farnell (none) -> 2059366
- R10, R23, R9: Farnell (none) -> 2502447
- R11, R12, R24: Farnell (none) -> 2059339
- R13, R14, R25: Farnell (none) -> 2059386
- R15, R16, R26: value 526R -> 562R; Farnell (none) -> 1170763
- R17, R18, R27: Farnell (none) -> 1170912
- R21, R22, R5, R6, R7, R8: Farnell (none) -> 1697388
- R28, R29, R30: Farnell (none) -> 9331662
- R31: Farnell (none) -> 2072517
- R32: Farnell (none) -> 2502502

Commit message: Final Tweaks before manufacture
Parts:
- removed C36: 100n, agg:0402-L, symbol C_Small
- removed R31: 10k, agg:0402-L, symbol R
Connections:
- net GND: now also IC10.4 (~EN)
Other:
- moved on the sheet: C35
