File: m3dl/pressure_relay/pressure_relay.kicad_pcb (KiCad board)
At the start: 2 copper layers, 40 x 33 mm, 13 parts, among them IC1 NCP380, IC2 ADuM1201, J1 WEST TOP, J2 EAST TOP, J3 WEST BOT, J4 UART, J5 EAST BOT, J6 SOUTH TOP, J7 SOUTH BOT

Commit message: Final changes to pressure relay
Parts:
- moved C2 0.76 mm to (91.3, 106.3), turned to 270 degrees
Routing:
- net GND: track 83.6 -> 240.9 mm, vias 12 -> 43
- net /3v3_FC: track 1.83 -> 3.31 mm
- net /3v3_PYRO: track 1.80 -> 3.25 mm
- net /3v3_DL: track 17.3 -> 18.7 mm
- net /PRESSURE2: track 17.3 -> 15.9 mm
- net /PRESSURE1: track 15.2 -> 16.3 mm
- net 3v3: track 31.3 -> 30.7 mm
Other:
- net class Default: clearance 0.2 -> 0.16; trace_width 0.2 -> 0.18
- rule trace_clearance: 0.2 -> 0.16
- rule trace_min: 0.2 -> 0.18
