File: m3dl/extpressure/extpressure.sch (KiCad schematic (older format))
At the start: 23 parts, among them IC1 SP100, IC2 SP100, IC3 SP100, IC4 SP100, IC5 STM32F0xxKxTx, J1 SERIAL, P1 SWD_TC

Commit message: ext pressure bom
Parts:
- C1, C2, C3, C4, C6, C7: Farnell (none) -> 2496771
- C5: Farnell (none) -> 2426952
- C8: Farnell (none) -> 2496814
- C9: Farnell (none) -> 2210793
- D1: Farnell (none) -> 2290329
- D2: Farnell (none) -> 2290328
- IC5: Farnell (none) -> 2333141
- J1: Farnell (none) -> 1830749
- R1, R2: Farnell (none) -> 2447120
Changed lines of the file:
@@
 EESchema Schematic File Version 2
-LIBS:agg-kicad
 LIBS:extpressure-cache
 EELAYER 25 0
@@
 F 2 "agg:LQFP-32" H 3200 3900 50  0001 L CNN
 F 3 "http://www.st.com/web/en/resource/technical/document/datasheet/DM00088500.pdf" H 3200 3800 50  0001 L CNN
+F 4 "2333141" H 3500 5100 60  0001 C CNN "Farnell"
 	1    3500 5100
 	1    0    0    -1
@@
 F 2 "agg:0402" H 2900 4350 50  0001 C CNN
 F 3 "" H 2900 4350 50  0001 C CNN
+F 4 "2210793" H 2900 4350 60  0001 C CNN "Farnell"
 	1    2900 4350
 	0    1    1    0
@@
 F 2 "agg:0402" H 2400 4250 50  0001 C CNN
 F 3 "" H 2400 4250 50  0001 C CNN
+F 4 "2496771" H 2400 4250 60  0001 C CNN "Farnell"
 	1    2400 4250
 	0    1    1    0
@@
 F 2 "agg:0402" H 2150 4150 50  0001 C CNN
 F 3 "" H 2150 4150 50  0001 C CNN
+F 4 "2496771" H 2150 4150 60  0001 C CNN "Farnell"
 	1    2150 4150
 	0    1    1    0
@@
 F 2 "agg:0402" H 2650 4350 50  0001 C CNN
 F 3 "" H 2650 4350 50  0001 C CNN
+F 4 "2496814" H 2650 4350 60  0001 C CNN "Farnell"
 	1    2650 4350
 	0    1    1    0
@@
 F 2 "agg:0402" H 1900 4150 50  0001 C CNN
 F 3 "" H 1900 4150 50  0001 C CNN
+F 4 "2426952" H 1900 4150 60  0001 C CNN "Farnell"
 	1    1900 4150
 	0    1    1    0
@@
 F 2 "agg:0402" H 1450 1750 50  0001 C CNN
 F 3 "" H 1450 1750 50  0001 C CNN
+F 4 "2496771" H 1450 1750 60  0001 C CNN "Farnell"
 	1    1450 1750
 	0    1    1    0
@@
 F 2 "agg:S04B-PASK-2" H 900 850 50  0001 C CNN
 F 3 "" H 900 850 50  0001 C CNN
+F 4 "1830749" H 900 850 60  0001 C CNN "Farnell"
 	1    900  850
 	1    0    0    -1
@@
 F 2 "agg:0603-LED" H 2650 5900 50  0001 C CNN
 F 3 "" H 2650 5900 50  0001 C CNN
+F 4 "2290329" H 2650 5900 60  0001 C CNN "Farnell"
 	1    2650 5900
 	1    0    0    1
@@
 F 2 "agg:0603-LED" H 4650 4500 50  0001 C CNN
 F 3 "" H 4650 4500 50  0001 C CNN
+F 4 "2290328" H 4650 4500 60  0001 C CNN "Farnell"
 	1    4650 4500
 	-1   0    0    1
@@
 F 2 "agg:0402" H 2550 5900 50  0001 C CNN
 F 3 "" H 2550 5900 50  0001 C CNN
+F 4 "2447120" H 2550 5900 60  0001 C CNN "Farnell"
 	1    2550 5900
 	-1   0    0    -1
@@
 F 2 "agg:0402" H 4750 4500 50  0001 C CNN
 F 3 "" H 4750 4500 50  0001 C CNN
+F 4 "2447120" H 4750 4500 60  0001 C CNN "Farnell"
 	1    4750 4500
 	1    0    0    -1
@@
 F 2 "agg:0402" H 3300 1750 50  0001 C CNN
 F 3 "" H 3300 1750 50  0001 C CNN
+F 4 "2496771" H 3300 1750 60  0001 C CNN "Farnell"
 	1    3300 1750
 	0    1    1    0
@@
 F 2 "agg:0402" H 5200 1750 50  0001 C CNN
 F 3 "" H 5200 1750 50  0001 C CNN
+F 4 "2496771" H 5200 1750 60  0001 C CNN "Farnell"
 	1    5200 1750
 	0    1    1    0
@@
 F 2 "agg:0402" H 7050 1750 50  0001 C CNN
 F 3 "" H 7050 1750 50  0001 C CNN
+F 4 "2496771" H 7050 1750 60  0001 C CNN "Farnell"
 	1    7050 1750
 	0    1    1    0
@@
 NoConn ~ 3100 6000
 $Comp
-L GND #PWR?
+L GND #PWR034
 U 1 1 5783A0D4
 P 4950 4550
-F 0 "#PWR?" H 4820 4590 50  0001 L CNN
+F 0 "#PWR034" H 4820 4590 50  0001 L CNN
 F 1 "GND" H 4950 4450 50  0000 C CNN
 F 2 "" H 4950 4550 60  0000 C CNN
