File: m3psu/pcb/DCDC-Board2/DCDC-Board2-Reg2.sch (KiCad schematic (older format))
At the start: 36 parts, among them IC2 LTC3887, Q3 SiZ340DT, Q4 SiZ340DT

Commit message: Added in ground pour on top side of DCDC board. DRC is not happy now...
Connections:
- net GND: no longer IC2.21 (PHAS_CFG)
- no-connect marks 5 -> 6
Changed lines of the file:
@@
 $EndComp
 $Comp
-L VCC #PWR041
+L VCC #PWR040
 U 1 1 56D586F4
 P 5150 1850
-F 0 "#PWR041" H 5150 1960 50  0001 L CNN
+F 0 "#PWR040" H 5150 1960 50  0001 L CNN
 F 1 "VCC" H 5150 1940 50  0000 C CNN
 F 2 "" H 5150 1850 60  0000 C CNN
@@
 $EndComp
 $Comp
-L GND #PWR042
+L GND #PWR041
 U 1 1 56D58702
 P 4850 2550
-F 0 "#PWR042" H 4720 2590 50  0001 L CNN
+F 0 "#PWR041" H 4720 2590 50  0001 L CNN
 F 1 "GND" H 4850 2450 50  0000 C CNN
 F 2 "" H 4850 2550 60  0000 C CNN
@@
 $EndComp
 $Comp
-L GND #PWR043
+L GND #PWR042
 U 1 1 56D58710
 P 5850 2200
-F 0 "#PWR043" H 5720 2240 50  0001 L CNN
+F 0 "#PWR042" H 5720 2240 50  0001 L CNN
 F 1 "GND" H 5850 2100 50  0000 C CNN
 F 2 "" H 5850 2200 60  0000 C CNN
@@
 $EndComp
 $Comp
-L GND #PWR044
+L GND #PWR043
 U 1 1 56D5873E
 P 7700 3100
-F 0 "#PWR044" H 7570 3140 50  0001 L CNN
+F 0 "#PWR043" H 7570 3140 50  0001 L CNN
 F 1 "GND" H 7700 3000 50  0000 C CNN
 F 2 "" H 7700 3100 60  0000 C CNN
@@
 $EndComp
 $Comp
-L GND #PWR045
+L GND #PWR044
 U 1 1 56D5874C
 P 4000 3100
-F 0 "#PWR045" H 3870 3140 50  0001 L CNN
+F 0 "#PWR044" H 3870 3140 50  0001 L CNN
 F 1 "GND" H 4000 3000 50  0000 C CNN
 F 2 "" H 4000 3100 60  0000 C CNN
@@
 $EndComp
 $Comp
-L GND #PWR046
+L GND #PWR045
 U 1 1 56D58772
 P 6600 4950
-F 0 "#PWR046" H 6470 4990 50  0001 L CNN
+F 0 "#PWR045" H 6470 4990 50  0001 L CNN
 F 1 "GND" H 6600 4850 50  0000 C CNN
 F 2 "" H 6600 4950 60  0000 C CNN
@@
 $EndComp
 $Comp
-L GND #PWR047
+L GND #PWR046
 U 1 1 56D58788
 P 5050 3500
-F 0 "#PWR047" H 4920 3540 50  0001 L CNN
+F 0 "#PWR046" H 4920 3540 50  0001 L CNN
 F 1 "GND" H 5050 3400 50  0000 C CNN
 F 2 "" H 5050 3500 60  0000 C CNN
@@
 $EndComp
 $Comp
-L GND #PWR048
+L GND #PWR047
 U 1 1 56D5878E
 P 4400 3200
-F 0 "#PWR048" H 4270 3240 50  0001 L CNN
+F 0 "#PWR047" H 4270 3240 50  0001 L CNN
 F 1 "GND" H 4400 3100 50  0000 C CNN
 F 2 "" H 4400 3200 60  0000 C CNN
@@
 $EndComp
 $Comp
-L GND #PWR049
+L GND #PWR048
 U 1 1 56D58794
 P 7300 3200
-F 0 "#PWR049" H 7170 3240 50  0001 L CNN
+F 0 "#PWR048" H 7170 3240 50  0001 L CNN
 F 1 "GND" H 7300 3100 50  0000 C CNN
 F 2 "" H 7300 3200 60  0000 C CNN
@@
 $EndComp
 $Comp
-L GND #PWR050
+L GND #PWR049
 U 1 1 56D587B2
 P 6850 2550
-F 0 "#PWR050" H 6720 2590 50  0001 L CNN
+F 0 "#PWR049" H 6720 2590 50  0001 L CNN
 F 1 "GND" H 6850 2450 50  0000 C CNN
 F 2 "" H 6850 2550 60  0000 C CNN
@@
 $EndComp
 $Comp
-L GND #PWR051
+L GND #PWR050
 U 1 1 56D587B8
 P 7350 4550
-F 0 "#PWR051" H 7220 4590 50  0001 L CNN
+F 0 "#PWR050" H 7220 4590 50  0001 L CNN
 F 1 "GND" H 7350 4450 50  0000 C CNN
 F 2 "" H 7350 4550 60  0000 C CNN
@@
 SCL
 $Comp
-L GND #PWR052
+L GND #PWR051
 U 1 1 56D587F8
 P 5050 4750
-F 0 "#PWR052" H 4920 4790 50  0001 L CNN
+F 0 "#PWR051" H 4920 4790 50  0001 L CNN
 F 1 "GND" H 5050 4650 50  0000 C CNN
 F 2 "" H 5050 4750 60  0000 C CNN
@@
 $EndComp
 $Comp
-L GND #PWR053
+L GND #PWR052
 U 1 1 56D58809
 P 6950 4300
-F 0 "#PWR053" H 6820 4340 50  0001 L CNN
+F 0 "#PWR052" H 6820 4340 50  0001 L CNN
 F 1 "GND" H 6950 4200 50  0000 C CNN
 F 2 "" H 6950 4300 60  0000 C CNN
@@
 $EndComp
 $Comp
-L GND #PWR054
+L GND #PWR053
 U 1 1 56D5881F
 P 7150 3650
-F 0 "#PWR054" H 7020 3690 50  0001 L CNN
+F 0 "#PWR053" H 7020 3690 50  0001 L CNN
 F 1 "GND" H 7150 3550 50  0000 C CNN
 F 2 "" H 7150 3650 60  0000 C CNN
@@
 $EndComp
 $Comp
-L GND #PWR055
+L GND #PWR054
 U 1 1 56D5883D
 P 4550 3750
-F 0 "#PWR055" H 4420 3790 50  0001 L CNN
+F 0 "#PWR054" H 4420 3790 50  0001 L CNN
 F 1 "GND" H 4550 3650 50  0000 C CNN
 F 2 "" H 4550 3750 60  0000 C CNN
@@
 	0    1    1    0
 $EndComp
-$Comp
-L GND #PWR056
-U 1 1 56D58843
-P 5100 5250
-F 0 "#PWR056" H 4970 5290 50  0001 L CNN
-F 1 "GND" H 5100 5150 50  0000 C CNN
-F 2 "" H 5100 5250 60  0000 C CNN
-F 3 "" H 5100 5250 60  0000 C CNN
-	1    5100 5250
-	1    0    0    -1
-$EndComp
-Wire Wire Line
-	5100 5200 5100 5250
 Wire Wire Line
 	7100 3650 7150 3650
@@
 Wire Wire Line
 	5050 4700 5050 4750
-Wire Wire Line
-	5100 5200 5150 5200
 Wire Wire Line
 	7250 4500 7350 4500
@@
 Connection ~ 5100 3500
 $Comp
-L GND #PWR057
+L GND #PWR055
 U 1 1 56D588E8
 P 6800 3500
-F 0 "#PWR057" H 6670 3540 50  0001 L CNN
+F 0 "#PWR055" H 6670 3540 50  0001 L CNN
 F 1 "GND" H 6800 3400 50  0000 C CNN
 F 2 "" H 6800 3500 60  0000 C CNN
@@
 $EndComp
 $Comp
-L GND #PWR058
+L GND #PWR056
 U 1 1 57476EC2
 P 5400 2200
-F 0 "#PWR058" H 5270 2240 50  0001 L CNN
+F 0 "#PWR056" H 5270 2240 50  0001 L CNN
 F 1 "GND" H 5400 2100 50  0000 C CNN
 F 2 "" H 5400 2200 60  0000 C CNN
@@
 	5200 2150 5150 2150
 Connection ~ 5150 2150
+NoConn ~ 5150 5200
 $EndSCHEMATC

Commit message: BOM for DCDC board 2 (inc swap 22u cap for in-stock)
Parts:
- C16, C22, C30: Farnell 1907510 -> 2346925
Changed lines of the file:
@@
 F 2 "agg:0805" H 5850 2050 50  0001 C CNN
 F 3 "" H 5850 2050 50  0001 C CNN
-F 4 "1907510" H 5850 2050 60  0001 C CNN "Farnell"
+F 4 "2346925" H 5850 2050 60  0001 C CNN "Farnell"
 	1    5850 2050
 	0    1    1    0
@@
 F 2 "agg:0805" H 7700 2950 50  0001 C CNN
 F 3 "" H 7700 2950 50  0001 C CNN
-F 4 "1907510" H 7700 2950 60  0001 C CNN "Farnell"
+F 4 "2346925" H 7700 2950 60  0001 C CNN "Farnell"
 	1    7700 2950
 	0    1    1    0
@@
 F 2 "agg:0805" H 4000 2950 50  0001 C CNN
 F 3 "" H 4000 2950 50  0001 C CNN
-F 4 "1907510" H 4000 2950 60  0001 C CNN "Farnell"
+F 4 "2346925" H 4000 2950 60  0001 C CNN "Farnell"
 	1    4000 2950
 	0    1    1    0

Commit message: routed one regulator
Parts:
- C19: footprint agg:0603 -> agg:0402; Farnell 2426959 -> 2346881
Changed lines of the file:
@@
 F 0 "C19" H 4900 2470 50  0000 C CNN
 F 1 "4µ7" H 4900 2330 50  0000 C CNN
-F 2 "agg:0603" H 4850 2400 50  0001 C CNN
+F 2 "agg:0402" H 4850 2400 50  0001 C CNN
 F 3 "" H 4850 2400 50  0001 C CNN
-F 4 "2426959" H 4850 2400 60  0001 C CNN "Farnell"
+F 4 "2346881" H 4850 2400 60  0001 C CNN "Farnell"
 	1    4850 2400
 	0    1    1    0
