File: m3psu/pcb/DCDC-Board1/DCDC-Board1.kicad_pcb (KiCad board)
At the start: 2 copper layers, 40 x 40 mm, 79 parts, among them IC1 LTC3887, IC2 LTC3887, J1 WEST TOP, J2 WEST BOT, J3 NORTH TOP, J4 EAST TOP, J5 EAST BOT, J6 NORTH BOT, Q1 SiZ340DT, Q2 SiZ340DT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

Commit message: improve silk and add gnd test point
Parts:
- added REF**: SIL-254P-01, agg:SIL-254P-01, F.Cu at (92.8, 85.1)
Other:
- board text added: "2016-07-25 JW LT AG"
- board text added: "M3PSU DCDC1"
- board text added: "r1"
- board text removed: "2016-07-25 r1 JW LT AG"
- board text removed: "M3PSU DCDC 1"
Changed lines of the file:
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@@
 (kicad_pcb (version 4) (host pcbnew 4.1.0-alpha+201605071002+6776~44~ubuntu14.04.1-product)
   (general
-    (links 272)
+    (links 0)
     (no_connects 0)
-    (area 79.899999 79.899999 120.100001 120.100001)
+    (area 79.899999 79.4575 120.1775 120.6775)
     (thickness 1.6)
-    (drawings 4)
+    (drawings 5)
     (tracks 1432)
     (zones 0)
-    (modules 79)
+    (modules 80)
     (nets 101)
   )
@@
     )
   )
-  (gr_text "2016-07-25\nr1 JW LT AG" (at 89.01 87.23 45) (layer F.SilkS)
+  (module agg:SIL-254P-01 (layer F.Cu)
+    (at 92.83 85.13 45)
+    (fp_text reference REF** (at 0 -2.22 45) (layer F.Fab)
+      (effects (font (size 1 1) (thickness 0.15)))
+    )
+    (fp_text value SIL-254P-01 (at 0 2.22 45) (layer F.Fab)
+      (effects (font (size 1 1) (thickness 0.15)))
+    )
+    (fp_line (start -1.27 -1.27) (end 1.27 -1.27) (layer F.Fab) (width 0.01))
+    (fp_line (start 1.27 -1.27) (end 1.27 1.27) (layer F.Fab) (width 0.01))
+    (fp_line (start 1.27 1.27) (end -1.27 1.27) (layer F.Fab) (width 0.01))
+    (fp_line (start -1.27 1.27) (end -1.27 -1.27) (layer F.Fab) (width 0.01))
+    (fp_line (start -1.27 -1.27) (end 1.27 -1.27) (layer F.SilkS) (width 0.15))
+    (fp_line (start 1.27 -1.27) (end 1.27 1.27) (layer F.SilkS) (width 0.15))
+    (fp_line (start 1.27 1.27) (end -1.27 1.27) (layer F.SilkS) (width 0.15))
+    (fp_line (start -1.27 1.27) (end -1.27 -1.27) (layer F.SilkS) (width 0.15))
+    (fp_line (start -1.55 -1.55) (end 1.55 -1.55) (layer F.CrtYd) (width 0.01))
+    (fp_line (start 1.55 -1.55) (end 1.55 1.55) (layer F.CrtYd) (width 0.01))
+    (fp_line (start 1.55 1.55) (end -1.55 1.55) (layer F.CrtYd) (width 0.01))
+    (fp_line (start -1.55 1.55) (end -1.55 -1.55) (layer F.CrtYd) (width 0.01))
+    (pad 1 thru_hole roundrect (at 0 0 45) (size 1.9 1.9) (drill 1) (layers *.Cu *.Mask F.SilkS)(roundrect_rratio 0.25)
+      (net 1 GND))
+    (model ${KISYS3DMOD}/Pin_Headers.3dshapes/Pin_Header_Straight_1x01.wrl
+      (at (xyz 0 0 0))
+      (scale (xyz 1 1 1))
+      (rotate (xyz 0 0 0))
+    )
+  )
+  (gr_text r1 (at 116.38 90.68 315) (layer F.SilkS)
     (effects (font (size 1.2 1.2) (thickness 0.25)))
   )
-  (gr_text "M3PSU\nDCDC 1" (at 108.31 84.83 315) (layer F.SilkS)
+  (gr_text "2016-07-25\nJW LT AG" (at 85 91.4 45) (layer F.SilkS)
+    (effects (font (size 1.2 1.2) (thickness 0.25)) (justify left))
+  )
+  (gr_text "M3PSU\nDCDC1" (at 108.31 84.83 315) (layer F.SilkS)
     (effects (font (size 1.2 1.2) (thickness 0.25)))
   )

Commit message: update DCDC address setting resistors due to making DCDC2 with DCDC1's resistors (intentionally)
Parts:
- R10: value 3k57 -> 5k76
- R23: value 4k32 -> 7k32
- R8: value 30k1 -> 24k9
Changed lines of the file:
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@@
-(kicad_pcb (version 4) (host pcbnew 4.1.0-alpha+201605071002+6776~44~ubuntu14.04.1-product)
+(kicad_pcb (version 4) (host pcbnew 0.201604290946+6713~44~ubuntu14.04.1-product)
   (general
-    (links 0)
+    (links 273)
     (no_connects 0)
-    (area 79.899999 79.4575 120.1775 120.6775)
+    (area 79.899999 79.899999 120.100001 120.100001)
     (thickness 1.6)
     (drawings 5)
@@
   )
   (setup
-    (last_trace_width 0.16)
+    (last_trace_width 0.25)
     (user_trace_width 0.16)
     (user_trace_width 0.2)
@@
       (effects (font (size 1 1) (thickness 0.15)))
     )
-    (fp_text value 4k32 (at 1.71 0 225) (layer F.Fab)
+    (fp_text value 7k32 (at 1.71 0 225) (layer F.Fab)
       (effects (font (size 1 1) (thickness 0.15)))
     )
@@
       (effects (font (size 1 1) (thickness 0.15)))
     )
-    (fp_text value 3k57 (at 1.71 0 225) (layer F.Fab)
+    (fp_text value 5k76 (at 1.71 0 225) (layer F.Fab)
       (effects (font (size 1 1) (thickness 0.15)))
     )
@@
       (effects (font (size 1 1) (thickness 0.15)))
     )
-    (fp_text value 30k1 (at 1.71 0 315) (layer F.Fab)
+    (fp_text value 24k9 (at 1.71 0 315) (layer F.Fab)
       (effects (font (size 1 1) (thickness 0.15)))
     )
@@
     )
   )
-  (module agg:SIL-254P-01 (layer F.Cu)
+  (module agg:SIL-254P-01 locked (layer F.Cu)
     (at 92.83 85.13 45)
     (fp_text reference REF** (at 0 -2.22 45) (layer F.Fab)
