File: m3radio/antennas/antennas.kicad_pcb (KiCad board)
At the start: 2 copper layers, 351.9 x 520.6 mm, 4 parts

Commit message: antennas r2 sent to manufacture
Parts:
- moved ? 8.59 mm to (195.9, 450.2)
- moved ? 6.19 mm to (89.1, 177.5)
- moved ? 5.19 mm to (195.9, 285.5)
Other:
- board size 351.9 x 520.6 mm -> 351.9 x 528.2 mm

Commit message: make smaller dart antenna cutouts to ease manufacture
Parts:
- moved ? 2.11 mm to (87.0, 25.0)
- moved ? 2.11 mm to (87.0, 177.5)
Other:
- outline, holes or cut-outs redrawn
