File: TOAD/TOAD.sch (KiCad schematic (older format))
At the start: 119 parts, among them IC1 MAX-M8Q, IC2 STM32F405RxTx, IC3 Si4463, IC4 BGS12AL7, IC5 Si4463, IC6 BGS12AL7, J1 USB, J6 SWITCH, P1 SWD_TC, P2 SMA, P3 SMA, P4 SMA, U1 MICROSD, X1 GPS ANT, X10 Power Switch, X11 RF Frame, X12 RF Cover, X2 USB Panel, X3 RF Frame, X4 RF Cover, X5 SMA Panel, X6 SMA Panel

Commit message: added clock buffer
Parts:
- added C?: 100n, agg:0603, symbol C_Small
- added IC?: SL18860DC, agg:DFN-10-SL18860DC, symbol SL18860DC
Connections:
- net 3v3: now also C?.1, IC?.2 (VDD), IC?.5 (OE3), IC?.6 (OE1), IC?.7 (OE2)
- net GND: now also C?.2, IC?.1 (VSS)
- net R_CLK_1: now also IC?.9 (CLKOUT2)
- net R_CLK_2: now also IC?.10 (CLKOUT3)
- net STM_HSE: now also IC?.8 (CLKOUT1)
- net VBATT: no longer J6.2
- net GATE: now reaches IC2.20 (PA4)
- net at IC?.3 (CLK_OUT): now also IC?.3 (CLKIN)
- net at J6.1: no longer J?.1
- no-connect marks 23 -> 34
Other:
- note added: "Clock Buffer"
- note added: "PLL to Remove Jitter from GPS Timepulse"
- note added: "Timepulse is set to 4MHz to act as the frequency\nreference for the system clock. PPS is set to produde \n1 pulse per second."
- note removed: "PLL to Remove Jitter from GPS"
- note removed: "SL18860DC"
- note removed: "Timepulse is set to 4MHz to feed the STM32 PLL, generating\na system clock of 144MHz and a periperal clock of 48MHz\nwith P=2, Q=6, M=4, N=288. Setting MCO1PRE to 5 produces\na 28.8MHz clock to feed to the Si4463."
- moved on the sheet: C?, IC?, J6, R?, Y?

Commit message: added PPS gating
Parts:
- added IC?: SN74LVC1G0832, agg:SC-70-6, symbol SN74LVC1G0832
Connections:
- net 3v3: now also IC?.5 (VCC)
- net GATE: now also IC?.3 (B)
- net GND: now also IC?.2 (GND)
- net GPS_PPS: now also IC?.1 (A)
- net PR_nSS: now also IC?.6 (C); no longer IC3.15 (nSEL)
- new net PR_CS: IC3.15 (nSEL), IC?.4 (Y)
Changed lines of the file:
@@
 SPI1_MISO
 Text Label 1800 2350 2    60   ~ 0
-PR_nSS
+PR_CS
 Text Label 1800 2050 2    60   ~ 0
 SPI1_SCK
@@
 NoConn ~ 3500 4200
 NoConn ~ 3500 4300
-Text Label 5000 2750 0    60   ~ 0
+Text Label 5650 2950 2    60   ~ 0
 PR_nSS
-Text Label 5000 2900 0    60   ~ 0
+Text Label 5650 2850 2    60   ~ 0
 GATE
-Text Label 5000 3050 0    60   ~ 0
+Text Label 5650 2750 2    60   ~ 0
 GPS_PPS
+$Comp
+L SN74LVC1G0832 IC?
+U 1 1 58BF7F01
+P 6050 2750
+F 0 "IC?" H 6050 3175 50  0000 C CNN
+F 1 "SN74LVC1G0832" H 6050 3084 50  0000 C CNN
+F 2 "agg:SC-70-6" H -500 -400 50  0001 L CNN
+F 3 "http://www.ti.com/lit/ds/symlink/sn74lvc1g0832.pdf" H -500 -500 50  0001 L CNN
+F 4 "2406965" H -500 -600 50  0001 L CNN "Farnell"
+	1    6050 2750
+	1    0    0    -1
+$EndComp
+Text Label 6450 2550 0    60   ~ 0
+PR_CS
+Wire Wire Line
+	6350 2750 6450 2750
+Wire Wire Line
+	6450 2750 6450 3000
+$Comp
+L GND #PWR?
+U 1 1 58BFC1CC
+P 6450 3000
+F 0 "#PWR?" H 6450 2750 50  0001 C CNN
+F 1 "GND" H 6450 2850 50  0000 C CNN
+F 2 "" H 6450 3000 50  0000 C CNN
+F 3 "" H 6450 3000 50  0000 C CNN
+	1    6450 3000
+	1    0    0    -1
+$EndComp
+Wire Wire Line
+	5750 2550 5650 2550
+Wire Wire Line
+	5650 2550 5650 2450
+$Comp
+L 3v3 #PWR?
+U 1 1 58BFC938
+P 5650 2450
+F 0 "#PWR?" H 5650 2560 50  0001 L CNN
+F 1 "3v3" H 5650 2540 50  0000 C CNN
+F 2 "" H 5650 2450 60  0000 C CNN
+F 3 "" H 5650 2450 60  0000 C CNN
+	1    5650 2450
+	-1   0    0    -1
+$EndComp
+Wire Wire Line
+	5650 2750 5750 2750
+Wire Wire Line
+	5650 2850 5750 2850
+Wire Wire Line
+	5650 2950 5750 2950
+Wire Wire Line
+	6350 2550 6450 2550
 $EndSCHEMATC

Commit message: added SDN and started charger but prioritised sleep over cusf
Parts:
- removed J6: SWITCH, agg:S02B-PASK-2, symbol CONN_01x02
- added C?: 1u, agg:0603, symbol C_Small
- added C? (x2): 4u7, agg:0603, symbol C_Small
- added J?: SWITCH, symbol CONN_01x03
Connections:
- net 5v: now also C?.1
- net B_TEMP: now also IC?.1 (TS)
- net GND: now also IC?.5 (EN2), C?.2, C?.2, C?.2, J?.3; no longer IC3.1 (SDN), IC5.1 (SDN)
- net VBATT: now also C?.1, J?.2
- net PR_SDN: now reaches IC2.2 (PC13)
- net PR_SDN: now also IC3.1 (SDN)
- net SR_SDN: now reaches IC2.3 (PC14)
- net SR_SDN: now also IC5.1 (SDN)
- net at IC?.10 (OUT): now also IC?.11 (OUT), IC?.6 (EN1)
- net P_GOOD: now reaches IC?.7 (~PGOOD)
- net CHG: now reaches IC?.9 (~CHG)
- net at C?.1, IC?.6 (SD), IC?.7 (IN)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: now also C?.1
- net at J?.1: now also J?.1
- no-connect marks 34 -> 32
Other:
- note added: "Primary Radio for Rocket TX/RX"
- note added: "Secondary Radio for TOAD Network Telemetry"
- note added: "Timepulse is set to 4MHz to act as the frequency\nreference for the system clock. PPS is set to produde \n1 pulse per second in falling mode."
- note removed: "Check 800mA Output\nSufficient"
- note removed: "Timepulse is set to 4MHz to act as the frequency\nreference for the system clock. PPS is set to produde \n1 pulse per second."
- moved on the sheet: C?, IC?, J1, J?, R1

Commit message: completed toad psu
Parts:
- added R?: 4k32, agg:0603-L, symbol R
- added R? (x2): 1M, agg:0603-L, symbol R
- added R? (x2): 10k, agg:0603-L, symbol R
- gave numbers to parts that had none: 39
- renumbered C31 to C1, C9 to C10, C6 to C11, C11 to C12, C16 to C13, C17 to C14, C22 to C15, C26 to C16, C2 to C17, C39 to C18, C3 to C19, C35 to C2, C29 to C20, C4 to C21, C7 to C22, C12 to C23, C13 to C27, C14 to C29, C38 to C3, C15 to C33, C18 to C34, C20 to C35, C1 to C36, C21 to C37, C23 to C38, C19 to C4, C24 to C45, C25 to C46, C27 to C47, C28 to C48, C30 to C49, C33 to C5, C32 to C50, C34 to C51, C36 to C53, C37 to C6, C8 to C7, C5 to C8, C10 to C9, D4 to D1, D2 to D10, D3 to D8, D1 to D9, IC3 to IC1, IC5 to IC10, IC6 to IC12, IC1 to IC2, IC2 to IC3, L8 to L1, L1 to L2, L9 to L3, L2 to L4, L3 to L5, L4 to L6, L5 to L7, L6 to L8, L7 to L9, P3 to P1, P1 to P2, P2 to P3, R10 to R16, R9 to R17, R2 to R3, R3 to R4, R4 to R5, R5 to R6, R6 to R7, R1 to R9, X3 to X2, X4 to X3, X2 to X4, X10 to X7, X11 to X8, X12 to X9
Connections:
- net 3v3: now also R?.2, R?.2
- net CHG: now also R?.1
- net GND: now also R?.1, R?.1
- net P_GOOD: now also R?.1
- net VBATT: now also R?.2
- net at IC7.10 (OUT), IC7.11 (OUT), IC7.6 (EN1): now also C32.1, C41.1, IC9.6 (SD), IC9.7 (IN), IC9.8 (IN)
- net I_CHG_MON: now reaches IC7.16 (ISET)
- net I_CHG_MON: now also R?.2
- net CHG_EN: now reaches IC7.4 (~CE)
- new net V_BAT_MON: R?.1, R?.2
- no-connect marks 32 -> 35
Other:
- note added: "TODO:\n- Hook up PSU to MCU\n- Check pin connections on all sections\n- Populate and confirm BOM\n- Add debug points \n- Begin PCB layout of each section\n- Investigate board size and physical layout\n- Solidworks model of layout\n- Complete PCB layout"
- moved on the sheet: C24, C25, C32, C41, C42, C44, IC7, IC9

Commit message: Completed STM32 section
Parts:
- removed C10: 100n, agg:0603, symbol C_Small
- removed C11: 100n, agg:0402, symbol C_Small
- added C13, C14: 100n, agg:0402, symbol C_Small
- C12, C4, C7, C8, C9: Farnell 2496834 -> 9402047
- R1, R2: symbol R -> R-RESCUE-TOAD; Farnell 2309108 -> 9238603
- R10: renamed from R7; symbol R -> R-RESCUE-TOAD
- R11, R12, R9: renamed from R?; symbol R -> R-RESCUE-TOAD
- R13: renamed from R8; symbol R -> R-RESCUE-TOAD
- R14: renamed from R9; symbol R -> R-RESCUE-TOAD
- R15: renamed from R10; symbol R -> R-RESCUE-TOAD
- R16: renamed from R11; symbol R -> R-RESCUE-TOAD
- R17: renamed from R12; symbol R -> R-RESCUE-TOAD
- R18: renamed from R13; symbol R -> R-RESCUE-TOAD
- R19: renamed from R14; symbol R -> R-RESCUE-TOAD
- R20: renamed from R15; symbol R -> R-RESCUE-TOAD
- R21: renamed from R16; symbol R -> R-RESCUE-TOAD
- R22: renamed from R17; symbol R -> R-RESCUE-TOAD
- R3: symbol R -> R-RESCUE-TOAD
- R4, R5: renamed from R?; value 1M -> 110k; symbol R -> R-RESCUE-TOAD
- R6: renamed from R4; symbol R -> R-RESCUE-TOAD
- R7: renamed from R5; symbol R -> R-RESCUE-TOAD
- R8: renamed from R6; symbol R -> R-RESCUE-TOAD
- X1, X4, X5, X6, X7: footprint Library:BMI-S-201-F -> (none)
- renumbered C13 to C10, C14 to C11, C26 to C24, C27 to C25, C28 to C26, C29 to C27, C30 to C28, C31 to C29, C33 to C30, C34 to C31, C35 to C32, C36 to C33, C37 to C34, C38 to C35, C32 to C36, C39 to C37, C40 to C38, C41 to C39, C24 to C40, C43 to C41, C25 to C42, C42 to C43, IC3 to IC1, IC9 to IC10, IC1 to IC2, IC2 to IC3, IC10 to IC9
Connections:
- net CHG is gone; now on net CHG_GOOD: IC7.9 (~CHG), R12.1
- net 3v3: now also C13.1, C14.1; no longer C7.1
- net B_TEMP: now also IC1.27 (PB1)
- net CHG_EN: now also IC1.28 (PB2)
- net GND: now also C7.1, C13.2, C14.2; no longer C7.2
- net I_CHG_MON: now also IC1.24 (PC4)
- net PR_SW: now also IC1.9 (PC1); no longer IC1.24 (PC4)
- net PR_nIRQ: now also IC1.30 (PB11); no longer IC1.25 (PC5)
- net P_GOOD: now also IC1.56 (PB4)
- net SR_nIRQ: now also IC1.4 (PC15); no longer IC1.9 (PC1)
- net V_BAT_MON: now also IC1.25 (PC5)
- net ~RST: now also C7.2
- net CHG_GOOD: now reaches IC1.55 (PB3)
- no-connect marks 35 -> 29
Other:
- note added: "ADC Channels:"
- note added: "ADC12_IN9/PB1 - B_TEMP\nADC12_IN14/PC4 - I_CHG_MON\nADC12_IN15/PC5 - V_BAT_MON"
- note added: "CH0 - Rsvd for TIM2 CH1\nCH1 - Rsvd for TIM2 CH2\nCH3/PB3 - CHG_GOOD\nCH4/PB4 - P_GOOD\nCH11/PB11 - PR_nIRQ\nCH15/PC15 - SR_nIRQ"
- note added: "Complete"
- note added: "Interrupt Channels:"
- note added: "TODO:\n- Check pin connections on all sections\n- Populate and confirm BOM\n- Add debug points \n- Begin PCB layout of each section\n- Investigate board size and physical layout\n- Solidworks model of layout\n- Complete PCB layout"
- note added: "Timer 2 (32-bit):"
- note added: "\nCH1/PA0 - GPS_PPS\nCH2/PA1 - PR_GPIO"
- note removed: "TODO:\n- Hook up PSU to MCU\n- Check pin connections on all sections\n- Populate and confirm BOM\n- Add debug points \n- Begin PCB layout of each section\n- Investigate board size and physical layout\n- Solidworks model of layout\n- Complete PCB layout"
- moved on the sheet: C10, C11, C15, C16, C4, C40, C42, IC1, P2, R1, R2

Commit message: Updated BOM and ERC
Parts:
- removed X6: SMA Panel, symbol PART
- added X12, X13, X8, X9: Mount, agg:M3_MOUNT, symbol PART
- added X3: Case, symbol PART
- added X4: SMA Panel, symbol PART
- added X7: Battery, symbol PART
- C10, C11, C16, C33, R10, R3, R6, R7, R8: footprint agg:0603 -> agg:0603-L
- C18: value 100nF -> 100n; footprint agg:0402 -> agg:0603-L; Farnell 1828860 -> 2496834
- C36, C42: footprint agg:0603 -> agg:0603-L; Farnell 2496834 -> 2496930
- C39, C40, C44: footprint agg:0603 -> agg:0603-L; Farnell 2496834 -> 1865556
- C43: footprint agg:0603 -> agg:0603-L; Farnell 2496834 -> 2496825
- D10, D3, D5, D7: Farnell 2290328 -> 2290329
- D2, D4, D6, D8: Farnell 2290329 -> 2290328
- IC3: Hab Supplies (none) -> HAB-MAX-M8Q
- J1: footprint agg:S04B-PASK-2 -> agg:SIL-254P-05; symbol CONN_01x04 -> CONN_01x05; RS (none) -> 841-8759
- J2, J3: footprint (none) -> agg:S03B-PASK-2; Farnell (none) -> 1830748
- P1: Farnell 1608592 -> (none); Hab Supplies (none) -> HAB-SL1252R
- R11, R12: value 10k -> 10K; Farnell 2309108 -> 9238603
- R15, R16, R17, R18, R19, R20, R21, R22: value 1k -> 120R; footprint agg:0603 -> agg:0603-L; Farnell 2309108 -> 9238379
- R4, R5: Farnell 2309108 -> 2502402
- R9: Farnell 2309108 -> 2670808
- X1: value GPS ANT -> USB Cap; Farnell 2497715 -> (none); RS (none) -> 123-6106
- X2: renamed from X4; value USB Panel -> USB Mini-B; Farnell 2497715 -> (none); RS (none) -> 252-438
- X5: Farnell 2497715 -> 2096227
- X6: renamed from X7; value Power Switch -> PWR Switch; Farnell 2497715 -> (none); RS (none) -> 123-6106
- renumbered X2 to X10, X3 to X11, X8 to X14, X9 to X15
Connections:
- net GND: now also J1.5; no longer IC2.5 (NC), IC9.5 (NC)
Other:
- note added: "External Parts:"
- note added: "PLL to Remove Jitter from GPS Frequency Reference"
- note added: "See /RangingSpecs.pdf for further notes"
- note removed: "PLL to Remove Jitter from GPS Timepulse"
- moved on the sheet: C37, J2, J3, R14, X2, X5, X6

Commit message: bom complete less radio passives
Parts:
- added D2, D3, D4, D5, D6, D7: ESD_DIODE, agg:0402-L, symbol ESD_DIODE
- C24, C28: footprint agg:0603 -> agg:0603-L; Farnell 2496834 -> 1865556
- C26: footprint agg:0603 -> agg:0603-L; Farnell 2496834 -> 2496825
- C29, C41, C52: footprint agg:0603 -> agg:0603-L
- C37, C38: footprint agg:0603 -> agg:0603-L; Farnell 2496834 -> 2496882
- R13: Farnell 2309108 -> 1469746
- Y1: footprint (none) -> agg:XTAL-25x20
- renumbered D4 to D10, D5 to D11, D6 to D12, D7 to D13, D9 to D14, D8 to D15, D10 to D16, D2 to D8, D3 to D9
Connections:
- net 5v: now also D2.1
- net B_TEMP: now also J2.2; no longer J2.3
- net GND: now also J2.3, D2.2, D3.2, D4.2, D5.2, D6.2, D7.2; no longer J2.2
- net OTG_HS_DM: now also D3.1
- net OTG_HS_DP: now also D4.1
- net VBATT: now also D5.1
- net at J2.1, J3.1: now also D6.1, D7.1
Other:
- moved on the sheet: D10, D11, D12, D13, D15, D16, D8, D9, J1, J2, J3, R14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

Commit message: Ready to begin PCB
Parts:
- removed C45: 3.9pF, agg:0402, symbol C_Small
- removed C46: 33pF, agg:0402, symbol C_Small
- removed C47: 8.2pF, agg:0402, symbol C_Small
- removed D14: ESD_DIODE, agg:0402-L, symbol ESD_DIODE
- added C24, C25, C54, C55, C56: DC, agg:0402, symbol C_Small
- added C30, C57, C59: 4.7pF, agg:0402, symbol C_Small
- added C52: 5.1pF, agg:0402, symbol C_Small
- added D15: ESD_DIODE, agg:0402-L, symbol ESD_DIODE
- C17: Farnell 2434643 -> 2524984
- C19: renamed from C20; Farnell 2434643 -> 2672775
- C20: renamed from C21; Farnell 2434643 -> 2133992
- C22: Farnell 2434643 -> 2688498
- C23: Farnell 2434643 -> 2672771
- C27: value 4.7pF -> DC; Farnell 2434643 -> (none)
- C28: renamed from C25; Farnell 2434643 -> 2332509
- C48: value 2.2pF -> 3pF; Farnell 2434643 -> 2524984
- C49: value 13pF -> 33pF
- C50: value 9.1pF -> 3.9pF; Farnell 2434643 -> 2672775
- C51: value 9.1pF -> 1pF; Farnell 2434643 -> 2133992
- C53: value 9.1pF -> 2.7pF; Farnell 2434643 -> 2672771
- L10: value 51nH -> 24nH; Farnell 1669580 -> 2470344
- L11: value 30nH -> 15nH; Farnell 1669580 -> 1762621
- L12: value 27nH -> 11nH; Farnell 1669580 -> 2116067
- L13: value 22nH -> 11nH; Farnell 1669580 -> 2116067
- L14: value 15nH -> 9.1nH; Farnell 1669580 -> 1762616
- L2: Farnell 1669580 -> 1748728
- L3: Farnell 1669580 -> 2470344
- L4: Farnell 1669580 -> 1762621
- L5, L6: Farnell 1669580 -> 2116067
- L7: Farnell 1669580 -> 1762616
- L8: value 220nH -> 120nH
- L9: value 56nH -> 20nH; Farnell 1669580 -> 1748728
- renumbered C19 to C18, C18 to C21, C24 to C26, C26 to C29, C28 to C31, C29 to C32, C30 to C33, C31 to C34, C32 to C35, C33 to C36, C34 to C37, C35 to C38, C36 to C39, C37 to C40, C38 to C41, C39 to C42, C40 to C43, C41 to C44, C42 to C45, C43 to C46, C44 to C47, C52 to C58, D15 to D14, IC5 to IC4, IC4 to IC5
Connections:
- net 3v3: now also C49.1
- net GND: now also C48.2, C49.2, C53.1, C30.2, C52.1, C57.2, C59.2, D15.2; no longer C27.2, C49.1, C50.1, C51.2, C53.2
- net SR_RXn: now also C48.1
- net SR_RXp: now also C51.1; no longer C48.1
- net SR_TX: now also C50.1
- net at C20.2, L3.2: now also C25.1; no longer IC5.1 (RF2)
- net at D1.1, L7.2, P3.1 (RF): now also C30.1; no longer C27.1
- net at IC5.3 (RF1): now also C24.2; no longer L6.2
- net at C28.1, L7.1: now also C27.2; no longer IC5.5 (RFIN)
- net at L11.1: now also C50.2
- net at L14.2, P4.1 (RF): now also C59.1, D15.1; no longer C53.1
- net at IC12.3 (RF1): now also C54.2; no longer L13.2
- net at L11.2, L12.1: now also C52.2; no longer C49.2
- net at L12.2, L13.1: now also C53.2; no longer C50.2
- new net: C25.2, IC5.1 (RF2)
- new net: C27.1, IC5.5 (RFIN)
- new net: C24.1, L6.2
- new net: C51.2, C55.1, L10.2
- new net: C55.2, IC12.1 (RF2)
- new net: C56.1, IC12.5 (RFIN)
- new net: C56.2, C57.1, L14.1
- new net: C54.1, L13.2
Other:
- note added: "TODO:\n- Add debug points \n- Begin PCB layout of each section\n- Place holes and board edge\n- Complete PCB layout"
- note removed: "Configured for 460MHz"
- note removed: "Incomplete"
- note removed: "TODO:\n- Check pin connections on all sections\n- Populate and confirm BOM\n- Add debug points \n- Begin PCB layout of each section\n- Investigate board size and physical layout\n- Solidworks model of layout\n- Complete PCB layout"
- moved on the sheet: C17, C18, C19, C20, C22, C23, C28, D1, IC5, L1, L2, L3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
