File: TOAD/TOAD.kicad_pcb (KiCad board)
At the start: 2 copper layers, 70 x 75 mm, 142 parts, among them IC1 STM32F405RxTx, IC10 ADP3335, IC11 CS2100-CP, IC12 BGS12AL7, IC13 SL18860DC, IC2 Si4463, IC3 MAX-M8Q, IC4 SN74LVC1G0832, IC5 BGS12AL7, IC6 ADP3335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

Commit message: pcb work
Parts:
- moved R6 86.2 mm to (45.7, 73.9)
- moved R10 83.0 mm to (50.4, 73.4)
- moved R7 77.2 mm to (43.4, 73.5)
- moved R1 75.2 mm to (85.8, 70.6), turned to 180 degrees
- moved R2 74.5 mm to (85.5, 72.8), turned to 180 degrees
- moved R3 67.9 mm to (53.1, 73.3)
- moved R8 67.9 mm to (47.8, 73.0)
- moved C36 60.5 mm to (59.7, 84.2), turned to 180 degrees
- moved R14 58.3 mm to (89.3, 82.4)
- moved R11 44.1 mm to (66.9, 141.1)
- moved IC10 41.9 mm to (78.1, 155.5)
- moved IC7 40.5 mm to (80.5, 147.3)
- moved C7 34.3 mm to (84.6, 104.2), turned to 270 degrees
- moved C42 33.9 mm to (72.5, 140.5)
- moved R5 28.6 mm to (60.1, 140.7)
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Routing:
- net GND: track 11.2 -> 15.4 mm
- net Net-(D6-Pad1): track 16.6 -> 20.4 mm
- net /B_TEMP: track 0.00 -> 2.15 mm
- net VBATT: track 0.00 -> 2.07 mm

Commit message: started psu layout for toad
Parts:
- moved IC7 42.3 mm to (73.0, 105.8)
- moved R7 26.1 mm to (68.5, 66.5)
- moved R8 19.8 mm to (66.5, 66.5)
- moved R6 18.4 mm to (62.5, 66.5)
- moved R3 13.3 mm to (64.5, 66.5)
- moved R10 12.2 mm to (60.5, 66.5)
- moved D5 0.45 mm to (65.3, 107.2)
Routing:
- net /B_TEMP: track 2.15 -> 34.6 mm
- net 5v: track 0.00 -> 23.5 mm
- net /SDIO_CMD: track 29.4 -> 42.7 mm
- net /SDIO_D2: track 26.6 -> 38.4 mm
- net /SDIO_D3: track 27.4 -> 37.9 mm
- net /SDIO_D0: track 0.00 -> 7.98 mm
- net VBATT: track 2.07 -> 8.91 mm
- net /SDIO_D1: track 0.00 -> 5.23 mm
- net GND: track 15.4 -> 13.3 mm
Changed lines of the file:
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@@
   (general
     (links 348)
-    (no_connects 204)
+    (no_connects 205)
     (area 35.385715 48.82 162.114286 159.108333)
     (thickness 1.6)
     (drawings 179)
-    (tracks 438)
+    (tracks 468)
     (zones 0)
     (modules 142)
@@
   )
   (setup
-    (last_trace_width 0.2)
+    (last_trace_width 0.25)
     (user_trace_width 0.15)
     (user_trace_width 0.2)
@@
   )
   (module agg:0402-L (layer F.Cu)
-    (at 65.3 106.8 270)
+    (at 65.3 107.25 270)
     (fp_text reference D5 (at -1.61 0) (layer F.Fab)
       (effects (font (size 1 1) (thickness 0.15)))
@@
   )
   (module agg:QFN-16-EP-TI (layer F.Cu)
-    (at 80.5 147.35)
+    (at 73 105.75)
     (fp_text reference IC7 (at 0 -2.65) (layer F.Fab)
       (effects (font (size 1 1) (thickness 0.15)))
@@
   )
   (module agg:0603-L (layer F.Cu)
-    (at 53.138047 73.319842 90)
+    (at 64.5 66.5 90)
     (fp_text reference R3 (at -2.025 0 180) (layer F.Fab)
       (effects (font (size 1 1) (thickness 0.15)))
@@
   )
   (module agg:0603-L (layer F.Cu)
-    (at 45.7 73.9 90)
+    (at 62.5 66.5 90)
     (fp_text reference R6 (at -2.025 0 180) (layer F.Fab)
       (effects (font (size 1 1) (thickness 0.15)))
@@
   )
   (module agg:0603-L (layer F.Cu)
-    (at 43.4 73.5 90)
+    (at 68.5 66.5 90)
     (fp_text reference R7 (at -2.025 0 180) (layer F.Fab)
       (effects (font (size 1 1) (thickness 0.15)))
@@
   )
   (module agg:0603-L (layer F.Cu)
-    (at 47.828047 72.969842 90)
+    (at 66.5 66.5 90)
     (fp_text reference R8 (at -2.025 0 180) (layer F.Fab)
       (effects (font (size 1 1) (thickness 0.15)))
@@
   )
   (module agg:0603-L (layer F.Cu)
-    (at 50.4 73.4 90)
+    (at 60.5 66.5 90)
     (fp_text reference R10 (at -2.6 -0.4 180) (layer F.Fab)
       (effects (font (size 1 1) (thickness 0.15)))
@@
   (segment (start 65.4 116.9) (end 64.1 116.9) (width 0.28) (layer F.Cu) (net 2))
   (segment (start 64.1 116.9) (end 63.5 117.5) (width 0.28) (layer F.Cu) (net 2))
-  (segment (start 65.3 107.2) (end 64.05 107.2) (width 0.28) (layer F.Cu) (net 2))
-  (segment (start 64.05 107.2) (end 63.5 107.75) (width 0.28) (layer F.Cu) (net 2))
   (via (at 97.5 123) (size 0.6) (drill 0.4) (layers F.Cu B.Cu) (net 2))
   (segment (start 97.5 123.8) (end 98.5 123.8) (width 0.35) (layer F.Cu) (net 2))
@@
   (segment (start 99.100971 71.035153) (end 99.500971 71.035153) (width 0.35) (layer F.Cu) (net 23))
   (segment (start 96.200971 71.035153) (end 96.900971 71.035153) (width 0.35) (layer F.Cu) (net 23))
-  (segment (start 63.5 105.75) (end 64.15 106.4) (width 0.28) (layer F.Cu) (net 25))
-  (segment (start 64.15 106.4) (end 65.3 106.4) (width 0.28) (layer F.Cu) (net 25))
+  (segment (start 67.5 88.67) (end 68.75 88.67) (width 0.28) (layer F.Cu) (net 24))
+  (segment (start 66 99.5) (end 66 90.17) (width 0.28) (layer F.Cu) (net 24))
+  (segment (start 66 90.17) (end 67.5 88.67) (width 0.28) (layer F.Cu) (net 24))
+  (segment (start 67.5 101) (end 66 99.5) (width 0.28) (layer F.Cu) (net 24))
+  (segment (start 72.25 101) (end 67.5 101) (width 0.28) (layer F.Cu) (net 24))
+  (segment (start 73.75 102.5) (end 72.25 101) (width 0.28) (layer F.Cu) (net 24))
+  (segment (start 73.75 104.35) (end 73.75 102.5) (width 0.28) (layer F.Cu) (net 24))
+  (segment (start 71.6 106) (end 71.25 106) (width 0.28) (layer F.Cu) (net 25))
+  (segment (start 71.25 106) (end 71 105.75) (width 0.28) (layer F.Cu) (net 25))
+  (segment (start 71.6 105.5) (end 71.25 105.5) (width 0.28) (layer F.Cu) (net 25))
+  (segment (start 71.25 105.5) (end 71 105.75) (width 0.28) (layer F.Cu) (net 25))
+  (segment (start 63.5 105.75) (end 71 105.75) (width 0.5) (layer F.Cu) (net 25))
   (segment (start 107.365 112.12) (end 107.365 112.91) (width 0.28) (layer F.Cu) (net 27))
   (segment (start 107.279228 112.995772) (end 107.365 112.91) (width 0.28) (layer F.Cu) (net 27))
@@
   (segment (start 116.025 109.9) (end 123.59 109.9) (width 1.06) (layer F.Cu) (net 39))
   (segment (start 122.55 109.9) (end 122.61 109.84) (width 0.28) (layer F.Cu) (net 39))
+  (segment (start 63.5 103.75) (end 60.5 103.75) (width 0.5) (layer F.Cu) (net 42))
+  (segment (start 60.5 113.5) (end 63.5 113.5) (width 0.5) (layer F.Cu) (net 42))
+  (segment (start 60.5 103.75) (end 59.5 104.75) (width 0.5) (layer F.Cu) (net 42))
+  (segment (start 59.5 104.75) (end 59.5 112.5) (width 0.5) (layer F.Cu) (net 42))
+  (segment (start 59.5 112.5) (end 60.5 113.5) (width 0.5) (layer F.Cu) (net 42))
   (segment (start 65.3 103.7) (end 63.55 103.7) (width 0.28) (layer F.Cu) (net 42))
   (segment (start 63.55 103.7) (end 63.5 103.75) (width 0.28) (layer F.Cu) (net 42))
   (segment (start 63.5 113.5) (end 65.5 113.5) (width 0.28) (layer F.Cu) (net 42))
-  (segment (start 59.5 104.75) (end 60.5 103.75) (width 0.8) (layer F.Cu) (net 42))
-  (segment (start 60.5 103.75) (end 63.5 103.75) (width 0.8) (layer F.Cu) (net 42))
-  (segment (start 59.5 112.5) (end 59.5 104.75) (width 0.8) (layer F.Cu) (net 42))
-  (segment (start 60.5 113.5) (end 59.5 112.5) (width 0.8) (layer F.Cu) (net 42))
-  (segment (start 63.5 113.5) (end 60.5 113.5) (width 0.8) (layer F.Cu) (net 42))
   (segment (start 86.5 118.7) (end 86.5 122.2) (width 0.28) (layer F.Cu) (net 43))
   (segment (start 88.5 118.7) (end 88.5 122.2) (width 0.28) (layer F.Cu) (net 44))
@@
   (segment (start 106.944228 89.39864) (end 107.144218 89.19865) (width 0.15) (layer F.Cu) (net 67))
   (segment (start 106.944228 90.02365) (end 106.944228 89.39864) (width 0.15) (layer F.Cu) (net 67))
+  (segment (start 60.25 115.5) (end 63.5 115.5) (width 0.25) (layer F.Cu) (net 71))
+  (segment (start 58.25 113.5) (end 60.25 115.5) (width 0.25) (layer F.Cu) (net 71))
+  (segment (start 58.25 103) (end 58.25 113.5) (width 0.25) (layer F.Cu) (net 71))
+  (segment (start 60.25 101) (end 58.25 103) (width 0.25) (layer F.Cu) (net 71))
+  (segment (start 65.25 101) (end 60.25 101) (width 0.25) (layer F.Cu) (net 71))
+  (segment (start 69.25 105) (end 65.25 101) (width 0.25) (layer F.Cu) (net 71))
+  (segment (start 71.6 105) (end 69.25 105) (width 0.25) (layer F.Cu) (net 71))
   (segment (start 65.4 116.1) (end 64.1 116.1) (width 0.28) (layer F.Cu) (net 71))
   (segment (start 64.1 116.1) (end 63.5 115.5) (width 0.28) (layer F.Cu) (net 71))
@@
   (segment (start 87.75 87.8) (end 87.75 89.65) (width 0.2) (layer F.Cu) (net 77))
   (segment (start 87.25 87.8) (end 87.25 89.15) (width 0.2) (layer F.Cu) (net 78))
+  (segment (start 64.5 70) (end 63.35 71.15) (width 0.25) (layer F.Cu) (net 79))
+  (segment (start 63.35 71.15) (end 59.8 71.15) (width 0.25) (layer F.Cu) (net 79))
+  (segment (start 64.5 67.2) (end 64.5 70) (width 0.25) (layer F.Cu) (net 79))
+  (segment (start 61.95 70.05) (end 62.5 69.5) (width 0.25) (layer F.Cu) (net 80))
+  (segment (start 62.5 69.5) (end 62.5 67.2) (width 0.25) (layer F.Cu) (net 80))
+  (segment (start 59.8 70.05) (end 61.95 70.05) (width 0.25) (layer F.Cu) (net 80))
   (segment (start 85.75 87.8) (end 85.75 89.15) (width 0.2) (layer F.Cu) (net 81))
   (segment (start 85.25 87.8) (end 85.25 89.75) (width 0.2) (layer F.Cu) (net 82))
@@
   (segment (start 76.760284 89.75) (end 80.3 89.75) (width 0.2) (layer F.Cu) (net 87))
   (segment (start 75.254523 85.945477) (end 75.254523 88.244239) (width 0.2) (layer F.Cu) (net 87))
+  (segment (start 68.5 67.2) (end 68.5 73.5) (width 0.25) (layer F.Cu) (net 89))
+  (segment (start 68.5 73.5) (end 64.6 77.4) (width 0.25) (layer F.Cu) (net 89))
   (segment (start 64.6 77.4) (end 64.6 78.19077) (width 0.25) (layer F.Cu) (net 89))
   (segment (start 64.6 78.19077) (end 77.15923 90.75) (width 0.25) (layer F.Cu) (net 89))
@@
   (via (at 61.35 77.65) (size 0.6) (drill 0.4) (layers F.Cu B.Cu) (net 89))
   (segment (start 59.8 77.65) (end 61.35 77.65) (width 0.25) (layer F.Cu) (net 89))
+  (segment (start 66.5 67.2) (end 66.5 73.9) (width 0.25) (layer F.Cu) (net 90))
+  (segment (start 66.5 73.9) (end 63.8 76.6) (width 0.25) (layer F.Cu) (net 90))
   (segment (start 61.4 76.6) (end 63.8 76.6) (width 0.25) (layer B.Cu) (net 90))
   (segment (start 63.8 76.6) (end 63.8 78.02718) (width 0.25) (layer F.Cu) (net 90))
@@
   (segment (start 63.05001 77.9136) (end 63.05001 74.25001) (width 0.25) (layer F.Cu) (net 91))
   (segment (start 63.05001 74.25001) (end 62.15 73.35) (width 0.25) (layer F.Cu) (net 91))
+  (segment (start 57 74.5) (end 57.95 75.45) (width 0.25) (layer F.Cu) (net 92))
+  (segment (start 57.95 75.45) (end 59.8 75.45) (width 0.25) (layer F.Cu) (net 92))
+  (segment (start 57 68.5) (end 57 74.5) (width 0.25) (layer F.Cu) (net 92))
+  (segment (start 58.3 67.2) (end 57 68.5) (width 0.25) (layer F.Cu) (net 92))
+  (segment (start 60.5 67.2) (end 58.3 67.2) (width 0.25) (layer F.Cu) (net 92))
   (segment (start 80.3 92.25) (end 76.75 92.25) (width 0.25) (layer F.Cu) (net 92))
   (segment (start 76.75 92.25) (end 62.6 78.1) (width 0.25) (layer F.Cu) (net 92))

Commit message: pcb progress
Parts:
- moved C43 47.0 mm to (71.5, 100.5)
- moved R9 45.3 mm to (70.0, 102.8), turned to 0 degrees
- moved R4 40.7 mm to (70.0, 107.5)
- moved IC10 40.3 mm to (73.0, 115.5), turned to 0 degrees
- moved C45 39.6 mm to (68.5, 107.5), turned to 270 degrees
- moved C39 38.4 mm to (76.5, 105.0)
- moved R5 32.0 mm to (70.0, 110.2)
- moved R11 31.4 mm to (72.7, 110.2), turned to 270 degrees
- moved R12 31.2 mm to (74.2, 110.2), turned to 270 degrees
- moved C46 29.6 mm to (73.0, 118.0), turned to 0 degrees
- moved C42 27.8 mm to (74.5, 112.8), turned to 180 degrees
- moved C47 26.8 mm to (68.8, 115.2), turned to 270 degrees
Routing:
- net 3v3: track 71.5 -> 151.0 mm, vias 4 -> 10
- net /P_GOOD: track 0.00 -> 33.3 mm, vias 0 -> 2
- net /CHG_GOOD: track 0.00 -> 30.8 mm, vias 0 -> 2
- net Net-(C39-Pad1): track 0.00 -> 19.5 mm, vias 0 -> 2
- net /B_TEMP: track 34.6 -> 20.7 mm, vias 0 -> 2
- net VBATT: track 8.91 -> 12.1 mm
- net /I_CHG_MON: track 0.00 -> 3.00 mm, vias 0 -> 1
- net Net-(C46-Pad2): track 0.00 -> 2.83 mm
- net /V_BAT_MON: track 0.00 -> 2.72 mm, vias 0 -> 1
- net Net-(C59-Pad1): track 10.7 -> 13.0 mm
- net Net-(C30-Pad1): track 8.63 -> 10.8 mm
- net GND: track 13.3 -> 15.1 mm
- net /CHG_EN: track 0.00 -> 1.21 mm, vias 0 -> 1
- net Net-(D17-Pad1): track 5.77 -> 6.95 mm
- added copper zone on F.Cu, net GND

Commit message: pcb work
Parts:
- moved C36 20.8 mm to (70.6, 66.5), turned to 270 degrees
- turned R10 to 270 degrees
Routing:
- net 3v3: track 151.0 -> 197.8 mm
- net /SDIO_CMD: track 42.7 -> 44.0 mm
Changed lines of the file:
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@@
   (general
     (links 348)
-    (no_connects 197)
+    (no_connects 88)
     (area 35.385715 48.82 162.114286 134.100001)
     (thickness 1.6)
     (drawings 179)
-    (tracks 606)
+    (tracks 624)
     (zones 0)
     (modules 142)
@@
   )
   (module agg:0603-L (layer F.Cu)
-    (at 59.7 84.2 180)
-    (fp_text reference C36 (at -2.025 0 270) (layer F.Fab)
+    (at 70.6 66.5 270)
+    (fp_text reference C36 (at -2.025 0) (layer F.Fab)
       (effects (font (size 1 1) (thickness 0.15)))
     )
-    (fp_text value 100n (at 2.025 0 270) (layer F.Fab)
+    (fp_text value 100n (at 2.025 0) (layer F.Fab)
       (effects (font (size 1 1) (thickness 0.15)))
     )
@@
     (fp_line (start 0.8 -0.4) (end 0.8 0.4) (layer F.Fab) (width 0.01))
     (fp_line (start -0.8 -0.4) (end 0.8 -0.4) (layer F.Fab) (width 0.01))
-    (pad 2 smd rect (at 0.7 0 180) (size 0.75 0.9) (layers F.Cu F.Paste F.Mask)
+    (pad 2 smd rect (at 0.7 0 270) (size 0.75 0.9) (layers F.Cu F.Paste F.Mask)
       (net 2 GND))
-    (pad 1 smd rect (at -0.7 0 180) (size 0.75 0.9) (layers F.Cu F.Paste F.Mask)
+    (pad 1 smd rect (at -0.7 0 270) (size 0.75 0.9) (layers F.Cu F.Paste F.Mask)
       (net 1 3v3))
     (model ${KISYS3DMOD}/Resistors_SMD.3dshapes/R_0603.wrl
@@
   )
   (module agg:0603-L (layer F.Cu)
-    (at 60.5 66.5 90)
-    (fp_text reference R10 (at -2.6 -0.4 180) (layer F.Fab)
+    (at 60.5 66.5 270)
+    (fp_text reference R10 (at -2.6 -0.4) (layer F.Fab)
       (effects (font (size 1 1) (thickness 0.15)))
     )
-    (fp_text value 47K (at 2.025 0 180) (layer F.Fab)
+    (fp_text value 47K (at 2.025 0) (layer F.Fab)
       (effects (font (size 1 1) (thickness 0.15)))
     )
@@
     (fp_line (start 0.8 -0.4) (end 0.8 0.4) (layer F.Fab) (width 0.01))
     (fp_line (start -0.8 -0.4) (end 0.8 -0.4) (layer F.Fab) (width 0.01))
-    (pad 2 smd rect (at 0.7 0 90) (size 0.75 0.9) (layers F.Cu F.Paste F.Mask)
+    (pad 2 smd rect (at 0.7 0 270) (size 0.75 0.9) (layers F.Cu F.Paste F.Mask)
       (net 1 3v3))
-    (pad 1 smd rect (at -0.7 0 90) (size 0.75 0.9) (layers F.Cu F.Paste F.Mask)
+    (pad 1 smd rect (at -0.7 0 270) (size 0.75 0.9) (layers F.Cu F.Paste F.Mask)
       (net 92 /SDIO_CMD))
     (model ${KISYS3DMOD}/Resistors_SMD.3dshapes/R_0603.wrl
@@
   (gr_line (start 60 130) (end 60 130) (layer Edge.Cuts) (width 0.1))
   (gr_line (start 130 130) (end 130 130) (layer Edge.Cuts) (width 0.1))
+  (segment (start 62.5 65.8) (end 62.2 65.8) (width 0.25) (layer F.Cu) (net 1))
+  (segment (start 62.2 65.8) (end 60.8 67.2) (width 0.25) (layer F.Cu) (net 1))
+  (segment (start 60.8 67.2) (end 60.5 67.2) (width 0.25) (layer F.Cu) (net 1))
+  (segment (start 57.6 68.1) (end 58.5 67.2) (width 0.25) (layer F.Cu) (net 1))
+  (segment (start 58.5 67.2) (end 60.5 67.2) (width 0.25) (layer F.Cu) (net 1))
+  (segment (start 57.6 73.8) (end 57.6 68.1) (width 0.25) (layer F.Cu) (net 1))
+  (segment (start 58.15 74.35) (end 57.6 73.8) (width 0.25) (layer F.Cu) (net 1))
+  (segment (start 59.8 74.35) (end 58.15 74.35) (width 0.25) (layer F.Cu) (net 1))
+  (segment (start 74.4 67.4) (end 72.8 65.8) (width 0.25) (layer F.Cu) (net 1))
+  (segment (start 72.8 65.8) (end 70.6 65.8) (width 0.25) (layer F.Cu) (net 1))
+  (segment (start 74.4 80.074998) (end 78.6 84.274998) (width 0.25) (layer F.Cu) (net 1))
+  (segment (start 74.4 80.074998) (end 74.4 67.4) (width 0.25) (layer F.Cu) (net 1))
+  (segment (start 77.050574 85.945477) (end 78.6 85.945477) (width 0.32) (layer F.Cu) (net 1))
+  (segment (start 78.6 85.945477) (end 80.254523 85.945477) (width 0.32) (layer F.Cu) (net 1))
+  (segment (start 78.6 84.274998) (end 78.6 85.945477) (width 0.25) (layer F.Cu) (net 1))
+  (segment (start 68.5 65.8) (end 70.6 65.8) (width 0.25) (layer F.Cu) (net 1))
+  (segment (start 68.5 65.8) (end 66.5 65.8) (width 0.25) (layer F.Cu) (net 1))
+  (segment (start 64.5 65.8) (end 66.5 65.8) (width 0.25) (layer F.Cu) (net 1))
+  (segment (start 62.5 65.8) (end 64.5 65.8) (width 0.25) (layer F.Cu) (net 1))
   (segment (start 82.05 102.15) (end 78.9 105.3) (width 0.5) (layer F.Cu) (net 1))
   (segment (start 78.9 105.3) (end 78.9 111.7) (width 0.5) (layer F.Cu) (net 1))
@@
   (segment (start 72.3 116.3) (end 72.3 118) (width 0.35) (layer F.Cu) (net 1))
   (segment (start 70.8 115.825) (end 71.825 115.825) (width 0.35) (layer F.Cu) (net 1))
-  (segment (start 77.050574 85.945477) (end 80.254523 85.945477) (width 0.32) (layer F.Cu) (net 1))
   (segment (start 80.254523 85.945477) (end 80.3 85.9) (width 0.32) (layer F.Cu) (net 1))
   (segment (start 92.35 89.75) (end 93.3 88.8) (width 0.25) (layer F.Cu) (net 1))
@@
   (segment (start 63.05001 77.9136) (end 63.05001 74.25001) (width 0.25) (layer F.Cu) (net 91))
   (segment (start 63.05001 74.25001) (end 62.15 73.35) (width 0.25) (layer F.Cu) (net 91))
+  (segment (start 57 67.2) (end 58.4 65.8) (width 0.25) (layer F.Cu) (net 92))
+  (segment (start 58.4 65.8) (end 60.5 65.8) (width 0.25) (layer F.Cu) (net 92))
+  (segment (start 57 74.5) (end 57 67.2) (width 0.25) (layer F.Cu) (net 92))
   (segment (start 57 74.5) (end 57.95 75.45) (width 0.25) (layer F.Cu) (net 92))
   (segment (start 57.95 75.45) (end 59.8 75.45) (width 0.25) (layer F.Cu) (net 92))
-  (segment (start 57 68.5) (end 57 74.5) (width 0.25) (layer F.Cu) (net 92))
-  (segment (start 58.3 67.2) (end 57 68.5) (width 0.25) (layer F.Cu) (net 92))
-  (segment (start 60.5 67.2) (end 58.3 67.2) (width 0.25) (layer F.Cu) (net 92))
   (segment (start 80.3 92.25) (end 76.75 92.25) (width 0.25) (layer F.Cu) (net 92))
   (segment (start 76.75 92.25) (end 62.6 78.1) (width 0.25) (layer F.Cu) (net 92))

Commit message: further pcb work, signal routing mostly complete
Parts:
- moved R1 6.73 mm to (87.7, 77.1), turned to 0 degrees
- moved R2 2.49 mm to (87.7, 74.0), turned to 0 degrees
- moved R14 2.42 mm to (90.3, 84.6), turned to 270 degrees
- moved C7 1.90 mm to (84.5, 102.3), turned to 90 degrees
- moved C13 1.02 mm to (94.3, 97.1), turned to 0 degrees
- moved D2 0.30 mm to (68.3, 86.2)
Routing:
- net /~RST: track 0.00 -> 55.6 mm, vias 0 -> 4
- net /USART1_RX: track 10.3 -> 63.9 mm, vias 0 -> 4
- net /SR_SW: track 0.00 -> 50.5 mm, vias 0 -> 2
- net /GPS_RST: track 0.00 -> 50.4 mm, vias 0 -> 4
- net /USART1_TX: track 9.01 -> 59.2 mm, vias 0 -> 4
- net /SR_ERR: track 0.00 -> 48.8 mm, vias 0 -> 2
- net /SR_GD: track 1.35 -> 47.4 mm, vias 0 -> 2
- net /PR_ERR: track 1.95 -> 44.5 mm, vias 0 -> 2
- net /PR_GD: track 1.35 -> 42.4 mm, vias 0 -> 2
- net /SDIO_D1: track 5.23 -> 44.4 mm, vias 0 -> 2
- net /SDIO_D0: track 7.98 -> 46.8 mm, vias 0 -> 2
- net /I2C1_SDA: track 2.93 -> 40.9 mm, vias 0 -> 2
- net /OTG_HS_DM: track 0.00 -> 37.4 mm, vias 0 -> 1
- net /PR_SW: track 0.00 -> 37.3 mm, vias 0 -> 4
- net /GPS_GD: track 1.35 -> 38.6 mm, vias 0 -> 2
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