File: m3psu/pcb/DCDC-5V/DCDC-5V.sch (KiCad schematic (older format))
At the start: 60 parts, among them IC1 LTC2975, IC2 TPS62133, IC3 TPS62152, J1 WEST TOP, J2 WEST BOT, J3 NORTH TOP, J4 EAST TOP, J5 EAST BOT, J6 NORTH BOT, Q1 NFET_GDS, Q2 NFET_GDS, Q3 NFET_GDS, Q4 NFET_GDS, Q5 PFET_GDS, Q6 PFET_GDS, Q7 PFET_GDS, Q8 PFET_GDS

Commit message: Complete BOM for DCDC-5V board
Parts:
- C1, C3, C4, C6: Farnell (none) -> 2496771
- C13, C8: Farnell (none) -> 1907510
- C2: Farnell (none) -> 1758924
- C5: Farnell (none) -> 2320856
- C7: Farnell (none) -> 1758918
- Q5, Q6, Q7, Q8: Farnell (none) -> 2501102
- R1: Farnell (none) -> 2670533
- R13, R14, R15, R16: Farnell (none) -> 2447160
- R17, R18, R19, R20: Farnell (none) -> RE05965
- R2, R3, R4, R5, R6, R7, R8: Farnell (none) -> 2447096
- R21, R22, R23, R24: Farnell (none) -> 2447127
Changed lines of the file:
@@
 F 2 "agg:0402" H 5400 5150 50  0001 C CNN
 F 3 "" H 5400 5150 50  0001 C CNN
+F 4 "2496771" H 5400 5150 60  0001 C CNN "Farnell"
 	1    5400 5150
 	0    1    1    0
@@
 F 2 "agg:0402" H 3450 4350 50  0001 C CNN
 F 3 "" H 3450 4350 50  0001 C CNN
+F 4 "2447096" H 3450 4350 60  0001 C CNN "Farnell"
 	1    3450 4350
 	1    0    0    -1
@@
 F 2 "agg:0402" H 3350 4450 50  0001 C CNN
 F 3 "" H 3350 4450 50  0001 C CNN
+F 4 "2447096" H 3350 4450 60  0001 C CNN "Farnell"
 	1    3350 4450
 	1    0    0    -1
@@
 F 2 "agg:0402" H 3450 4550 50  0001 C CNN
 F 3 "" H 3450 4550 50  0001 C CNN
+F 4 "2447096" H 3450 4550 60  0001 C CNN "Farnell"
 	1    3450 4550
 	1    0    0    -1
@@
 F 2 "agg:0402" H 3350 4650 50  0001 C CNN
 F 3 "" H 3350 4650 50  0001 C CNN
+F 4 "2447096" H 3350 4650 60  0001 C CNN "Farnell"
 	1    3350 4650
 	1    0    0    -1
@@
 F 2 "agg:0402" H 3500 3650 50  0001 C CNN
 F 3 "" H 3500 3650 50  0001 C CNN
+F 4 "2447096" H 3500 3650 60  0001 C CNN "Farnell"
 	1    3500 3650
 	1    0    0    -1
@@
 F 2 "agg:0402" H 3350 3550 50  0001 C CNN
 F 3 "" H 3350 3550 50  0001 C CNN
+F 4 "2447096" H 3350 3550 60  0001 C CNN "Farnell"
 	1    3350 3550
 	1    0    0    -1
@@
 F 2 "agg:0402" H 3500 3450 50  0001 C CNN
 F 3 "" H 3500 3450 50  0001 C CNN
+F 4 "2447096" H 3500 3450 60  0001 C CNN "Farnell"
 	1    3500 3450
 	1    0    0    -1
@@
 F 2 "agg:0402" H 3450 2850 50  0001 C CNN
 F 3 "" H 3450 2850 50  0001 C CNN
+F 4 "1758924" H 3450 2850 60  0001 C CNN "Farnell"
 	1    3450 2850
 	1    0    0    -1
@@
 F 2 "agg:0402" H 3450 3150 50  0001 C CNN
 F 3 "" H 3450 3150 50  0001 C CNN
+F 4 "2496771" H 3450 3150 60  0001 C CNN "Farnell"
 	1    3450 3150
 	1    0    0    -1
@@
 F 2 "agg:0402" H 3250 1950 50  0001 C CNN
 F 3 "" H 3250 1950 50  0001 C CNN
+F 4 "2496771" H 3250 1950 60  0001 C CNN "Farnell"
 	1    3250 1950
 	1    0    0    -1
@@
 F 2 "agg:0402" H 6900 1050 50  0001 C CNN
 F 3 "" H 6900 1050 50  0001 C CNN
+F 4 "2447160" H 6900 1050 60  0001 C CNN "Farnell"
 	1    6900 1050
 	0    1    1    0
@@
 F 2 "agg:0603" H 7150 1550 50  0001 C CNN
 F 3 "" H 7150 1550 50  0001 C CNN
+F 4 "RE05965" H 7150 1550 60  0001 C CNN "Farnell"
 	1    7150 1550
 	0    -1   -1   0
@@
 F 2 "agg:0402" H 6900 2550 50  0001 C CNN
 F 3 "" H 6900 2550 50  0001 C CNN
+F 4 "2447160" H 6900 2550 60  0001 C CNN "Farnell"
 	1    6900 2550
 	0    1    1    0
@@
 F 2 "agg:0603" H 7150 3050 50  0001 C CNN
 F 3 "" H 7150 3050 50  0001 C CNN
+F 4 "RE05965" H 7150 3050 60  0001 C CNN "Farnell"
 	1    7150 3050
 	0    -1   -1   0
@@
 F 2 "agg:0402" H 6900 4050 50  0001 C CNN
 F 3 "" H 6900 4050 50  0001 C CNN
+F 4 "2447160" H 6900 4050 60  0001 C CNN "Farnell"
 	1    6900 4050
 	0    1    1    0
@@
 F 2 "agg:0603" H 7150 4550 50  0001 C CNN
 F 3 "" H 7150 4550 50  0001 C CNN
+F 4 "RE05965" H 7150 4550 60  0001 C CNN "Farnell"
 	1    7150 4550
 	0    -1   -1   0
@@
 F 2 "agg:0402" H 6900 5550 50  0001 C CNN
 F 3 "" H 6900 5550 50  0001 C CNN
+F 4 "2447160" H 6900 5550 60  0001 C CNN "Farnell"
 	1    6900 5550
 	0    1    1    0
@@
 F 2 "agg:0603" H 7150 6050 50  0001 C CNN
 F 3 "" H 7150 6050 50  0001 C CNN
+F 4 "RE05965" H 7150 6050 60  0001 C CNN "Farnell"
 	1    7150 6050
 	0    -1   -1   0
@@
 F 2 "agg:SON2x2" H 7150 1150 50  0001 C CNN
 F 3 "" H 7150 1150 50  0001 C CNN
+F 4 "2501102" V 7150 1150 60  0001 C CNN "Farnell"
 	1    7150 1150
 	1    0    0    -1
@@
 F 2 "agg:SON2x2" H 7150 2650 50  0001 C CNN
 F 3 "" H 7150 2650 50  0001 C CNN
+F 4 "2501102" V 7150 2650 60  0001 C CNN "Farnell"
 	1    7150 2650
 	1    0    0    -1
@@
 F 2 "agg:SON2x2" H 7150 4150 50  0001 C CNN
 F 3 "" H 7150 4150 50  0001 C CNN
+F 4 "2501102" V 7150 4150 60  0001 C CNN "Farnell"
 	1    7150 4150
 	1    0    0    -1
@@
 F 2 "agg:SON2x2" H 7150 5650 50  0001 C CNN
 F 3 "" H 7150 5650 50  0001 C CNN
+F 4 "2501102" V 7150 5650 60  0001 C CNN "Farnell"
 	1    7150 5650
 	1    0    0    -1
@@
 F 2 "agg:0402" H 1300 1650 50  0001 C CNN
 F 3 "" H 1300 1650 50  0001 C CNN
+F 4 "1758918" H 1300 1650 60  0001 C CNN "Farnell"
 	1    1300 1650
 	0    1    1    0
@@
 F 2 "agg:0402" H 1150 1350 50  0001 C CNN
 F 3 "" H 1150 1350 50  0001 C CNN
+F 4 "2496771" H 1150 1350 60  0001 C CNN "Farnell"
 	1    1150 1350
 	0    1    1    0
@@
 F 2 "agg:0805" H 950 1650 50  0001 C CNN
 F 3 "" H 950 1650 50  0001 C CNN
+F 4 "2320856" H 950 1650 60  0001 C CNN "Farnell"
 	1    950  1650
 	0    1    1    0
@@
 F 2 "agg:0805" H 2800 1300 50  0001 C CNN
 F 3 "" H 2800 1300 50  0001 C CNN
+F 4 "1907510" H 2800 1300 60  0001 C CNN "Farnell"
 	1    2800 1300
 	0    1    1    0
@@
 F 2 "agg:0402" H 3500 2450 50  0001 C CNN
 F 3 "" H 3500 2450 50  0001 C CNN
+F 4 "2670533" H 3500 2450 60  0001 C CNN "Farnell"
 	1    3500 2450
 	1    0    0    -1
@@
 F 2 "agg:0402" H 6650 1550 50  0001 C CNN
 F 3 "" H 6650 1550 50  0001 C CNN
+F 4 "2447127" H 6650 1550 60  0001 C CNN "Farnell"
 	1    6650 1550
 	0    1    1    0
@@
 F 2 "agg:0402" H 6650 3050 50  0001 C CNN
 F 3 "" H 6650 3050 50  0001 C CNN
+F 4 "2447127" H 6650 3050 60  0001 C CNN "Farnell"
 	1    6650 3050
 	0    1    1    0
@@
 F 2 "agg:0402" H 6650 4550 50  0001 C CNN
 F 3 "" H 6650 4550 50  0001 C CNN
+F 4 "2447127" H 6650 4550 60  0001 C CNN "Farnell"
 	1    6650 4550
 	0    1    1    0
@@
 F 2 "agg:0402" H 6650 6050 50  0001 C CNN
 F 3 "" H 6650 6050 50  0001 C CNN
+F 4 "2447127" H 6650 6050 60  0001 C CNN "Farnell"
 	1    6650 6050
 	0    1    1    0
@@
 F 2 "agg:0805" H 3050 1300 50  0001 C CNN
 F 3 "" H 3050 1300 50  0001 C CNN
+F 4 "1907510" H 3050 1300 60  0001 C CNN "Farnell"
 	1    3050 1300
 	0    1    1    0
