File: m3psu/pcb/DCDC-3V/DCDC-3V.sch (KiCad schematic (older format))
At the start: 68 parts, among them IC1 LTC2975, IC2 TPS62132, IC3 LTC2975, J1 WEST TOP, J2 WEST BOT, J3 NORTH TOP, J4 EAST TOP, J5 EAST BOT, J6 NORTH BOT, Q1 NFET_GDS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

Commit message: Update NFET footprint, add VEN pull-downs
Parts:
- added R35, R36, R37, R38, R39, R40: 1M, agg:0402, symbol R
- C5: value 10µ -> 10u
- C8: value 22µ -> 22u
- L1: value 2µ2 -> 2u2
- Q1, Q11, Q2, Q3, Q4, Q9: footprint agg:SOT-883-B -> agg:PowerPAK-SC-75-6L-Single; Farnell (none) -> 2364070
- Q10, Q12, Q5, Q6, Q7, Q8: Farnell (none) -> 2501102
- R10, R11, R12, R29, R32, R9: Fit (none) -> NOFIT
Connections:
- net GND: now also R35.2, R36.2, R37.2, R38.2, R39.2, R40.2
- net VEN_0: now also R35.1
- net VEN_1: now also R36.1
- net VEN_2: now also R37.1
- net VEN_3: now also R38.1
- net VEN_4: now also R39.1
- net VEN_5: now also R40.1
- no-connect marks 15 -> 16

Commit message: Add test pads, decoupling capacitor to 3V board
Parts:
- added C13: 22u, agg:0805, symbol C
- added TP1, TP2, TP3, TP4: TESTPAD, agg:TESTPAD, symbol TESTPAD
Connections:
- net 3v3: now also C13.1
- net GND: now also C13.2, TP4.1 (TP)
- net SCL: now also TP2.1 (TP)
- net SDA: now also TP1.1 (TP)
- net ~ALERT: now also TP3.1 (TP)
Other:
- note added: "TEST POINTS"

Commit message: Complete BOM for DCDC-3V board
Parts:
- C1, C11, C12, C3, C4, C6, C9: Farnell (none) -> 2496771
- C10, C2: Farnell (none) -> 1758924
- C13, C8: Farnell (none) -> 1907510
- C5: Farnell (none) -> 2320856
- C7: Farnell (none) -> 1758918
- J3: Samtec (none) -> TFML-105-02-L-D
- J6: Samtec (none) -> SFML-105-02-L-D-LC
- R1, R26: Farnell (none) -> 2670533
- R13, R14, R15, R16, R30, R33: Farnell (none) -> 2447160
- R17, R18, R19, R20, R31, R34: Farnell (none) -> RE05965
- R2, R21, R22, R23, R24, R25, R27, R28, R3, R4, R5, R6, R7, R8: Farnell (none) -> 2447096
- R35, R36, R37, R38, R39, R40: Farnell (none) -> 2447127
Changed lines of the file:
@@
 F 2 "agg:TFML-105-02-L-D" H 9000 3300 50  0001 C CNN
 F 3 "" H 9000 3300 50  0001 C CNN
+F 4 "TFML-105-02-L-D" H 9000 3300 60  0001 C CNN "Samtec"
 	1    9000 3300
 	1    0    0    -1
@@
 F 2 "agg:SFML-105-02-L-D-LC" H 10400 3300 50  0001 C CNN
 F 3 "" H 10400 3300 50  0001 C CNN
+F 4 "SFML-105-02-L-D-LC" H 10400 3300 60  0001 C CNN "Samtec"
 	1    10400 3300
 	1    0    0    -1
@@
 F 2 "agg:0402" H 5600 6500 50  0001 C CNN
 F 3 "" H 5600 6500 50  0001 C CNN
+F 4 "2496771" H 5600 6500 60  0001 C CNN "Farnell"
 	1    5600 6500
 	0    1    1    0
@@
 F 2 "agg:0402" H 3650 5700 50  0001 C CNN
 F 3 "" H 3650 5700 50  0001 C CNN
+F 4 "2447096" H 3650 5700 60  0001 C CNN "Farnell"
 	1    3650 5700
 	1    0    0    -1
@@
 F 2 "agg:0402" H 3550 5800 50  0001 C CNN
 F 3 "" H 3550 5800 50  0001 C CNN
+F 4 "2447096" H 3550 5800 60  0001 C CNN "Farnell"
 	1    3550 5800
 	1    0    0    -1
@@
 F 2 "agg:0402" H 3650 5900 50  0001 C CNN
 F 3 "" H 3650 5900 50  0001 C CNN
+F 4 "2447096" H 3650 5900 60  0001 C CNN "Farnell"
 	1    3650 5900
 	1    0    0    -1
@@
 F 2 "agg:0402" H 3550 6000 50  0001 C CNN
 F 3 "" H 3550 6000 50  0001 C CNN
+F 4 "2447096" H 3550 6000 60  0001 C CNN "Farnell"
 	1    3550 6000
 	1    0    0    -1
@@
 F 2 "agg:0402" H 3700 5000 50  0001 C CNN
 F 3 "" H 3700 5000 50  0001 C CNN
+F 4 "2447096" H 3700 5000 60  0001 C CNN "Farnell"
 	1    3700 5000
 	1    0    0    -1
@@
 F 2 "agg:0402" H 3550 4900 50  0001 C CNN
 F 3 "" H 3550 4900 50  0001 C CNN
+F 4 "2447096" H 3550 4900 60  0001 C CNN "Farnell"
 	1    3550 4900
 	1    0    0    -1
@@
 F 2 "agg:0402" H 3700 4800 50  0001 C CNN
 F 3 "" H 3700 4800 50  0001 C CNN
+F 4 "2447096" H 3700 4800 60  0001 C CNN "Farnell"
 	1    3700 4800
 	1    0    0    -1
@@
 F 2 "agg:0402" H 3650 4200 50  0001 C CNN
 F 3 "" H 3650 4200 50  0001 C CNN
+F 4 "1758924" H 3650 4200 60  0001 C CNN "Farnell"
 	1    3650 4200
 	1    0    0    -1
@@
 F 2 "agg:0402" H 3650 4500 50  0001 C CNN
 F 3 "" H 3650 4500 50  0001 C CNN
+F 4 "2496771" H 3650 4500 60  0001 C CNN "Farnell"
 	1    3650 4500
 	1    0    0    -1
@@
 F 2 "agg:0402" H 3450 3300 50  0001 C CNN
 F 3 "" H 3450 3300 50  0001 C CNN
+F 4 "2496771" H 3450 3300 60  0001 C CNN "Farnell"
 	1    3450 3300
 	1    0    0    -1
@@
 F 2 "agg:0402" H 6850 950 50  0001 C CNN
 F 3 "" H 6850 950 50  0001 C CNN
+F 4 "2447160" H 6850 950 60  0001 C CNN "Farnell"
 	1    6850 950
 	0    1    1    0
@@
 F 2 "agg:0603" H 7100 1450 50  0001 C CNN
 F 3 "" H 7100 1450 50  0001 C CNN
+F 4 "RE05965" H 7100 1450 60  0001 C CNN "Farnell"
 	1    7100 1450
 	0    -1   -1   0
@@
 F 2 "agg:0402" H 6850 2450 50  0001 C CNN
 F 3 "" H 6850 2450 50  0001 C CNN
+F 4 "2447160" H 6850 2450 60  0001 C CNN "Farnell"
 	1    6850 2450
 	0    1    1    0
@@
 F 2 "agg:0603" H 7100 2950 50  0001 C CNN
 F 3 "" H 7100 2950 50  0001 C CNN
+F 4 "RE05965" H 7100 2950 60  0001 C CNN "Farnell"
 	1    7100 2950
 	0    -1   -1   0
@@
 F 2 "agg:0402" H 6850 3950 50  0001 C CNN
 F 3 "" H 6850 3950 50  0001 C CNN
+F 4 "2447160" H 6850 3950 60  0001 C CNN "Farnell"
 	1    6850 3950
 	0    1    1    0
@@
 F 2 "agg:0603" H 7100 4450 50  0001 C CNN
 F 3 "" H 7100 4450 50  0001 C CNN
+F 4 "RE05965" H 7100 4450 60  0001 C CNN "Farnell"
 	1    7100 4450
 	0    -1   -1   0
@@
 F 2 "agg:0402" H 6850 5450 50  0001 C CNN
 F 3 "" H 6850 5450 50  0001 C CNN
+F 4 "2447160" H 6850 5450 60  0001 C CNN "Farnell"
 	1    6850 5450
 	0    1    1    0
@@
 F 2 "agg:0603" H 7100 5950 50  0001 C CNN
 F 3 "" H 7100 5950 50  0001 C CNN
+F 4 "RE05965" H 7100 5950 60  0001 C CNN "Farnell"
 	1    7100 5950
 	0    -1   -1   0
@@
 F 2 "agg:0402" H 4050 1700 50  0001 C CNN
 F 3 "" H 4050 1700 50  0001 C CNN
+F 4 "1758918" H 4050 1700 60  0001 C CNN "Farnell"
 	1    4050 1700
 	0    1    1    0
@@
 F 2 "agg:0402" H 3900 1400 50  0001 C CNN
 F 3 "" H 3900 1400 50  0001 C CNN
+F 4 "2496771" H 3900 1400 60  0001 C CNN "Farnell"
 	1    3900 1400
 	0    1    1    0
@@
 F 2 "agg:0805" H 3700 1700 50  0001 C CNN
 F 3 "" H 3700 1700 50  0001 C CNN
+F 4 "2320856" H 3700 1700 60  0001 C CNN "Farnell"
 	1    3700 1700
 	0    1    1    0
@@
 F 2 "agg:0805" H 5550 1350 50  0001 C CNN
 F 3 "" H 5550 1350 50  0001 C CNN
+F 4 "1907510" H 5550 1350 60  0001 C CNN "Farnell"
 	1    5550 1350
 	0    1    1    0
@@
 F 2 "agg:0402" H 3700 3800 50  0001 C CNN
 F 3 "" H 3700 3800 50  0001 C CNN
+F 4 "2670533" H 3700 3800 60  0001 C CNN "Farnell"
 	1    3700 3800
 	1    0    0    -1
@@
 F 2 "agg:0402" H 8550 5450 50  0001 C CNN
 F 3 "" H 8550 5450 50  0001 C CNN
+F 4 "2447160" H 8550 5450 60  0001 C CNN "Farnell"
 	1    8550 5450
 	0    1    1    0
@@
 F 2 "agg:0603" H 8800 5950 50  0001 C CNN
 F 3 "" H 8800 5950 50  0001 C CNN
+F 4 "RE05965" H 8800 5950 60  0001 C CNN "Farnell"
 	1    8800 5950
 	0    -1   -1   0
@@
 F 2 "agg:0402" H 10250 5450 50  0001 C CNN
 F 3 "" H 10250 5450 50  0001 C CNN
+F 4 "2447160" H 10250 5450 60  0001 C CNN "Farnell"
 	1    10250 5450
 	0    1    1    0
@@
 F 2 "agg:0603" H 10500 5950 50  0001 C CNN
 F 3 "" H 10500 5950 50  0001 C CNN
+F 4 "RE05965" H 10500 5950 60  0001 C CNN "Farnell"
 	1    10500 5950
 	0    -1   -1   0
@@
 F 2 "agg:0402" H 2900 4150 50  0001 C CNN
 F 3 "" H 2900 4150 50  0001 C CNN
+F 4 "2496771" H 2900 4150 60  0001 C CNN "Farnell"
 	1    2900 4150
 	0    1    1    0
@@
 F 2 "agg:0402" H 950 3350 50  0001 C CNN
 F 3 "" H 950 3350 50  0001 C CNN
+F 4 "2447096" H 950 3350 60  0001 C CNN "Farnell"
 	1    950  3350
 	1    0    0    -1
@@
 F 2 "agg:0402" H 850 3450 50  0001 C CNN
 F 3 "" H 850 3450 50  0001 C CNN
+F 4 "2447096" H 850 3450 60  0001 C CNN "Farnell"
 	1    850  3450
 	1    0    0    -1
@@
 F 2 "agg:0402" H 950 3550 50  0001 C CNN
 F 3 "" H 950 3550 50  0001 C CNN
+F 4 "2447096" H 950 3550 60  0001 C CNN "Farnell"
 	1    950  3550
 	1    0    0    -1
@@
 F 2 "agg:0402" H 850 3650 50  0001 C CNN
 F 3 "" H 850 3650 50  0001 C CNN
+F 4 "2447096" H 850 3650 60  0001 C CNN "Farnell"
 	1    850  3650
 	1    0    0    -1
@@
 F 2 "agg:0402" H 1000 2650 50  0001 C CNN
 F 3 "" H 1000 2650 50  0001 C CNN
+F 4 "2447096" H 1000 2650 60  0001 C CNN "Farnell"
 	1    1000 2650
 	1    0    0    -1
@@
 F 2 "agg:0402" H 850 2550 50  0001 C CNN
 F 3 "" H 850 2550 50  0001 C CNN
+F 4 "2447096" H 850 2550 60  0001 C CNN "Farnell"
 	1    850  2550
 	1    0    0    -1
@@
 F 2 "agg:0402" H 1000 2450 50  0001 C CNN
 F 3 "" H 1000 2450 50  0001 C CNN
+F 4 "2447096" H 1000 2450 60  0001 C CNN "Farnell"
 	1    1000 2450
 	1    0    0    -1
@@
 F 2 "agg:0402" H 950 1850 50  0001 C CNN
 F 3 "" H 950 1850 50  0001 C CNN
+F 4 "1758924" H 950 1850 60  0001 C CNN "Farnell"
 	1    950  1850
 	1    0    0    -1
@@
 F 2 "agg:0402" H 950 2150 50  0001 C CNN
 F 3 "" H 950 2150 50  0001 C CNN
+F 4 "2496771" H 950 2150 60  0001 C CNN "Farnell"
 	1    950  2150
 	1    0    0    -1
@@
 F 2 "agg:0402" H 750 950 50  0001 C CNN
 F 3 "" H 750 950 50  0001 C CNN
+F 4 "2496771" H 750 950 60  0001 C CNN "Farnell"
 	1    750  950
 	1    0    0    -1
@@
 F 2 "agg:0402" H 1000 1450 50  0001 C CNN
 F 3 "" H 1000 1450 50  0001 C CNN
+F 4 "2670533" H 1000 1450 60  0001 C CNN "Farnell"
 	1    1000 1450
 	1    0    0    -1
@@
 F 2 "agg:0402" H 6600 1450 50  0001 C CNN
 F 3 "" H 6600 1450 50  0001 C CNN
+F 4 "2447127" H 6600 1450 60  0001 C CNN "Farnell"
 	1    6600 1450
 	0    1    1    0
@@
 F 2 "agg:0402" H 6600 2950 50  0001 C CNN
 F 3 "" H 6600 2950 50  0001 C CNN
+F 4 "2447127" H 6600 2950 60  0001 C CNN "Farnell"
 	1    6600 2950
 	0    1    1    0
@@
 F 2 "agg:0402" H 6600 4450 50  0001 C CNN
 F 3 "" H 6600 4450 50  0001 C CNN
+F 4 "2447127" H 6600 4450 60  0001 C CNN "Farnell"
 	1    6600 4450
 	0    1    1    0
@@
 F 2 "agg:0402" H 6600 5950 50  0001 C CNN
 F 3 "" H 6600 5950 50  0001 C CNN
+F 4 "2447127" H 6600 5950 60  0001 C CNN "Farnell"
 	1    6600 5950
 	0    1    1    0
@@
 F 2 "agg:0402" H 8300 5950 50  0001 C CNN
 F 3 "" H 8300 5950 50  0001 C CNN
+F 4 "2447127" H 8300 5950 60  0001 C CNN "Farnell"
 	1    8300 5950
 	0    1    1    0
@@
 F 2 "agg:0402" H 10000 5950 50  0001 C CNN
 F 3 "" H 10000 5950 50  0001 C CNN
+F 4 "2447127" H 10000 5950 60  0001 C CNN "Farnell"
 	1    10000 5950
 	0    1    1    0
@@
 F 2 "agg:0805" H 5800 1350 50  0001 C CNN
 F 3 "" H 5800 1350 50  0001 C CNN
+F 4 "1907510" H 5800 1350 60  0001 C CNN "Farnell"
 	1    5800 1350
 	0    1    1    0
